File: main_board/B.B/_saved_power.sch (KiCad schematic (older format))
At the start: 36 parts, among them Q1 CJ3134K, Q2 CJ3134K, U62 AOZ1280, U63 FP6296

Commit message: orezavani
smazaní A9G, SD karty, a zvuku
Parts:
- removed L1: 2.2uH, BB:SMD-PIND-10.5x11.5x4_2.5x3.0, symbol Device:L
- added L?: 3.3uH, BB:SMD-PIND-12.8x13.5x5_2.0x5.0, symbol Device:L
Connections:
- net 3V3: now also L?.2
- net at C85.1, D1.1 (K), U62.6 (LX): now also L?.1
Changed lines of the file:
@@
-$EndComp
-$Comp
-L Device:L L1
-U 1 1 5FA64342
-P 7500 2250
-F 0 "L1" V 7690 2250 50  0000 C CNN
-F 1 "2.2uH" V 7599 2250 50  0000 C CNN
-F 2 "BB:SMD-PIND-10.5x11.5x4_2.5x3.0" H 7500 2250 50  0001 C CNN
-F 3 "~" H 7500 2250 50  0001 C CNN
-F 4 "C149550" V 7500 2250 50  0001 C CNN "LCSC"
-	1    7500 2250
-	0    -1   -1   0
 $EndComp
 $Comp
@@
 	1    0    0    -1
 $EndComp
+$Comp
+L Device:L L?
+U 1 1 5FBDFC00
+P 7500 2250
+F 0 "L?" V 7690 2250 50  0000 C CNN
+F 1 "3.3uH" V 7599 2250 50  0000 C CNN
+F 2 "BB:SMD-PIND-12.8x13.5x5_2.0x5.0" H 7500 2250 50  0001 C CNN
+F 3 "~" H 7500 2250 50  0001 C CNN
+F 4 "C149571" V 7500 2250 50  0001 C CNN "LCSC"
+	1    7500 2250
+	0    -1   -1   0
+$EndComp
 $EndSCHEMATC
