File: main_board/B.B/B.B.sch (KiCad schematic (older format))
At the start: 9 parts

Commit message: konzultace_s_Kubou_01
Parts:
- removed R? (x2): 12k, Resistor_SMD:R_0402_1005Metric, symbol Device:R
- added R? (x2): 7.5k, Resistor_SMD:R_0402_1005Metric, symbol Device:R
Changed lines of the file:
@@
 Wire Wire Line
 	5800 2050 7050 2050
-$Comp
-L Device:R R?
-U 1 1 5F9AE21A
-P 6750 1750
-F 0 "R?" H 6820 1796 50  0000 L CNN
-F 1 "12k" H 6820 1705 50  0000 L CNN
-F 2 "Resistor_SMD:R_0402_1005Metric" V 6680 1750 50  0001 C CNN
-F 3 "~" H 6750 1750 50  0001 C CNN
-F 4 "C25752" H 6750 1750 50  0001 C CNN "LCSC"
-	1    6750 1750
-	1    0    0    -1
-$EndComp
 Wire Wire Line
 	6750 1600 6750 1550
@@
 Wire Wire Line
 	6750 1950 7150 1950
-$Comp
-L Device:R R?
-U 1 1 5F9B8EBB
-P 7050 1750
-F 0 "R?" H 7120 1796 50  0000 L CNN
-F 1 "12k" H 7120 1705 50  0000 L CNN
-F 2 "Resistor_SMD:R_0402_1005Metric" V 6980 1750 50  0001 C CNN
-F 3 "~" H 7050 1750 50  0001 C CNN
-F 4 "C25752" H 7050 1750 50  0001 C CNN "LCSC"
-	1    7050 1750
-	1    0    0    -1
-$EndComp
 Wire Wire Line
 	7050 1600 7050 1550
@@
 F18 "ENC_OUT_0" I L 7600 4500 50
 F19 "ENC_OUT_1" I L 7600 4600 50
+F20 "IO1_3" I R 8600 4000 50
+F21 "MOTOR" I R 8600 3900 50
 $EndSheet
 Wire Wire Line
@@
 Wire Wire Line
 	7600 4500 5800 4500
+$Comp
+L Device:R R?
+U 1 1 5FA54DFA
+P 6750 1750
+AR Path="/5FA4C94D/5FA54DFA" Ref="R?"  Part="1"
+AR Path="/5F9AAC80/5FA54DFA" Ref="R?"  Part="1"
+AR Path="/5FA54DFA" Ref="R?"  Part="1"
+F 0 "R?" V 6650 1750 50  0000 C CNN
+F 1 "7.5k" V 6850 1750 50  0000 C CNN
+F 2 "Resistor_SMD:R_0402_1005Metric" V 6680 1750 50  0001 C CNN
+F 3 "~" H 6750 1750 50  0001 C CNN
+F 4 "C25918" H 6750 1750 50  0001 C CNN "LCSC"
+	1    6750 1750
+	-1   0    0    1
+$EndComp
+$Comp
+L Device:R R?
+U 1 1 5FA57DCC
+P 7050 1750
+AR Path="/5FA4C94D/5FA57DCC" Ref="R?"  Part="1"
+AR Path="/5F9AAC80/5FA57DCC" Ref="R?"  Part="1"
+AR Path="/5FA57DCC" Ref="R?"  Part="1"
+F 0 "R?" V 6950 1750 50  0000 C CNN
+F 1 "7.5k" V 7150 1750 50  0000 C CNN
+F 2 "Resistor_SMD:R_0402_1005Metric" V 6980 1750 50  0001 C CNN
+F 3 "~" H 7050 1750 50  0001 C CNN
+F 4 "C25918" H 7050 1750 50  0001 C CNN "LCSC"
+	1    7050 1750
+	-1   0    0    1
+$EndComp
 $EndSCHEMATC

Commit message: preparation_to_drawing_PCB
Parts:
- removed J?: Conn_01x03, symbol Connector_Generic:Conn_01x03
- removed R? (x2): 20k, symbol Device:R
- removed R?: 5.6k, symbol Device:R
- added J?: Conn_01x02, symbol Connector_Generic:Conn_01x02
- added R?: 1M, Resistor_SMD:R_0402_1005Metric, symbol Device:R
- R?: value 12k -> 330k; footprint (none) -> Capacitor_SMD:C_0402_1005Metric; LCSC C25752 -> C25778
Connections:
- net labels removed: +4V, BateriMiddle, SHUTDOWN_4V
- wire segments 98 -> 95
Other:
- moved on the sheet: R?

Commit message: complete_preparation_to_drawing_PCB
footprint for all component and LCSC code for everything for mounting in JLCPCB
Parts:
- J1: renamed from J?; footprint (none) -> Connector_PinHeader_2.54mm:PinHeader_1x02_P2.54mm_Vertical
- J2, J3: renamed from J?; footprint (none) -> Connector_PinHeader_2.54mm:PinHeader_1x08_P2.54mm_Vertical
- gave numbers to parts that had none: 4
Changed lines of the file:
@@
 	7050 3600 7600 3600
 $Comp
-L B.B-eagle-import:VCC #V?
+L B.B-eagle-import:VCC #V01
 U 1 1 5FA8B2FC
 P 2550 1250
-F 0 "#V?" H 2550 1250 50  0001 C CNN
+F 0 "#V01" H 2550 1250 50  0001 C CNN
 F 1 "VCC" H 2550 1380 59  0000 C CNN
 F 2 "" H 2550 1250 50  0001 C CNN
@@
 	2550 1450 2800 1450
 $Comp
-L B.B-eagle-import:VCC #V?
+L B.B-eagle-import:VCC #V06
 U 1 1 5FA8BF43
 P 4500 2000
-F 0 "#V?" H 4500 2000 50  0001 C CNN
+F 0 "#V06" H 4500 2000 50  0001 C CNN
 F 1 "VCC" H 4500 2130 59  0000 C CNN
 F 2 "" H 4500 2000 50  0001 C CNN
@@
 $EndComp
 $Comp
-L Device:R R?
+L Device:R R4
 U 1 1 5FA8E393
 P 4500 2550
-F 0 "R?" H 4570 2596 50  0000 L CNN
+F 0 "R4" H 4570 2596 50  0000 L CNN
 F 1 "330k" H 4570 2505 50  0000 L CNN
 F 2 "Capacitor_SMD:C_0402_1005Metric" V 4430 2550 50  0001 C CNN
@@
 $EndComp
 $Comp
-L B.B-eagle-import:GND #GND?
+L B.B-eagle-import:GND #GND061
 U 1 1 5FA8F1DF
 P 2300 1750
-F 0 "#GND?" H 2300 1750 50  0001 C CNN
+F 0 "#GND061" H 2300 1750 50  0001 C CNN
 F 1 "GND" H 2300 1670 59  0000 C CNN
 F 2 "" H 2300 1750 50  0001 C CNN
@@
 $EndComp
 $Comp
-L B.B-eagle-import:GND #GND?
+L B.B-eagle-import:GND #GND062
 U 1 1 5FA8F578
 P 4500 2800
-F 0 "#GND?" H 4500 2800 50  0001 C CNN
+F 0 "#GND062" H 4500 2800 50  0001 C CNN
 F 1 "GND" H 4500 2720 59  0000 C CNN
 F 2 "" H 4500 2800 50  0001 C CNN
@@
 	3500 1650 4000 1650
 $Comp
-L B.B-eagle-import:+5V #V?
+L B.B-eagle-import:+5V #V02
 U 1 1 5F96BCF7
 P 3600 1300
-F 0 "#V?" H 3600 1300 50  0001 C CNN
+F 0 "#V02" H 3600 1300 50  0001 C CNN
 F 1 "+5V" H 3600 1430 59  0000 C CNN
 F 2 "" H 3600 1300 50  0001 C CNN
@@
 $EndComp
 $Comp
-L B.B-eagle-import:+3V3 #V?
+L B.B-eagle-import:+3V3 #V03
 U 1 1 5F96C236
 P 4000 1300
-F 0 "#V?" H 4000 1300 50  0001 C CNN
+F 0 "#V03" H 4000 1300 50  0001 C CNN
 F 1 "+3V3" H 4000 1430 59  0000 C CNN
 F 2 "" H 4000 1300 50  0001 C CNN
@@
 	4000 1650 4800 1650
 $Comp
-L B.B-eagle-import:+5V #V?
+L B.B-eagle-import:+5V #V05
 U 1 1 5F970ABB
 P 7500 1300
-F 0 "#V?" H 7500 1300 50  0001 C CNN
+F 0 "#V05" H 7500 1300 50  0001 C CNN
 F 1 "+5V" H 7500 1430 59  0000 C CNN
 F 2 "" H 7500 1300 50  0001 C CNN
@@
 $EndComp
 $Comp
-L B.B-eagle-import:+3V3 #V?
+L B.B-eagle-import:+3V3 #V04
 U 1 1 5F9711C3
 P 6750 1300
-F 0 "#V?" H 6750 1300 50  0001 C CNN
+F 0 "#V04" H 6750 1300 50  0001 C CNN
 F 1 "+3V3" H 6750 1430 59  0000 C CNN
 F 2 "" H 6750 1300 50  0001 C CNN
@@
 SHUTDOWN_3V3
 $Sheet
-S 8800 5150 550  950
+S 8550 5150 550  950
 U 5FA9675D
 F0 "next-board00" 50
 F1 "next-board.sch" 50
-F2 "SCL" I L 8800 5450 50
-F3 "SDA" I L 8800 5550 50
-F4 "INT" I L 8800 5700 50
-F5 "SHUTDOWN" I L 8800 5850 50
-F6 "3V3" I L 8800 5300 50
-F7 "WS2812" I L 8800 6000 50
-F8 "5V" I L 8800 5200 50
+F2 "SCL" I L 8550 5450 50
+F3 "SDA" I L 8550 5550 50
+F4 "INT" I L 8550 5700 50
+F5 "SHUTDOWN" I L 8550 5850 50
+F6 "3V3" I L 8550 5300 50
+F7 "WS2812" I L 8550 6000 50
+F8 "5V" I L 8550 5200 50
 $EndSheet
 $Comp
-L Connector_Generic:Conn_01x08 J?
+L Connector_Generic:Conn_01x08 J2
 U 1 1 60051102
 P 7800 5450
-F 0 "J?" V 7900 5700 50  0000 L CNN
+F 0 "J2" V 7900 5700 50  0000 L CNN
 F 1 "Conn_01x08" V 7900 4950 50  0000 L CNN
-F 2 "" H 7800 5450 50  0001 C CNN
+F 2 "Connector_PinHeader_2.54mm:PinHeader_1x08_P2.54mm_Vertical" H 7800 5450 50  0001 C CNN
 F 3 "~" H 7800 5450 50  0001 C CNN
 	1    7800 5450
@@
 $EndComp
 $Comp
-L Connector_Generic:Conn_01x08 J?
+L Connector_Generic:Conn_01x08 J3
 U 1 1 600527FF
 P 8000 5450
-F 0 "J?" V 8100 5700 50  0000 L CNN
+F 0 "J3" V 8100 5700 50  0000 L CNN
 F 1 "Conn_01x08" V 8100 4950 50  0000 L CNN
-F 2 "" H 8000 5450 50  0001 C CNN
+F 2 "Connector_PinHeader_2.54mm:PinHeader_1x08_P2.54mm_Vertical" H 8000 5450 50  0001 C CNN
 F 3 "~" H 8000 5450 50  0001 C CNN
 	1    8000 5450
@@
 	8300 5250 8300 5200
 Wire Wire Line
-	8300 5200 8800 5200
-Wire Wire Line
-	8200 5350 8650 5350
-Wire Wire Line
-	8650 5350 8650 5300
-Wire Wire Line
-	8650 5300 8800 5300
+	8300 5200 8550 5200
+Wire Wire Line
+	8200 5350 8500 5350
+Wire Wire Line
+	8500 5350 8500 5300
+Wire Wire Line
+	8500 5300 8550 5300
 Wire Wire Line
 	8200 5150 8300 5150
@@
 Connection ~ 8300 5200
 Wire Wire Line
-	8200 5450 8800 5450
-Wire Wire Line
-	8800 5550 8200 5550
-Wire Wire Line
-	8750 5650 8750 5700
-Wire Wire Line
-	8750 5700 8800 5700
-Wire Wire Line
-	8200 5650 8750 5650
-Wire Wire Line
-	8800 5850 8650 5850
-Wire Wire Line
-	8650 5850 8650 5750
-Wire Wire Line
-	8650 5750 8200 5750
-Wire Wire Line
-	8200 5850 8550 5850
-Wire Wire Line
-	8550 5850 8550 6000
-Wire Wire Line
-	8550 6000 8800 6000
+	8200 5450 8550 5450
+Wire Wire Line
+	8550 5550 8200 5550
+Wire Wire Line
+	8500 5650 8500 5700
+Wire Wire Line
+	8500 5700 8550 5700
+Wire Wire Line
+	8200 5650 8500 5650
+Wire Wire Line
+	8550 5850 8400 5850
+Wire Wire Line
+	8400 5850 8400 5750
+Wire Wire Line
+	8400 5750 8200 5750
+Wire Wire Line
+	8200 5850 8300 5850
+Wire Wire Line
+	8300 5850 8300 6000
+Wire Wire Line
+	8300 6000 8550 6000
 Wire Wire Line
 	7500 5250 7600 5250
@@
 AR Path="/5FA4C94D/5FA54DFA" Ref="R?"  Part="1"
 AR Path="/5F9AAC80/5FA54DFA" Ref="R?"  Part="1"
-AR Path="/5FA54DFA" Ref="R?"  Part="1"
-F 0 "R?" V 6650 1750 50  0000 C CNN
+AR Path="/5FA54DFA" Ref="R1"  Part="1"
+F 0 "R1" V 6650 1750 50  0000 C CNN
 F 1 "7.5k" V 6850 1750 50  0000 C CNN
 F 2 "Resistor_SMD:R_0402_1005Metric" V 6680 1750 50  0001 C CNN
@@
 AR Path="/5FA4C94D/5FA57DCC" Ref="R?"  Part="1"
 AR Path="/5F9AAC80/5FA57DCC" Ref="R?"  Part="1"
-AR Path="/5FA57DCC" Ref="R?"  Part="1"
-F 0 "R?" V 6950 1750 50  0000 C CNN
+AR Path="/5FA57DCC" Ref="R2"  Part="1"
+F 0 "R2" V 6950 1750 50  0000 C CNN
 F 1 "7.5k" V 7150 1750 50  0000 C CNN
 F 2 "Resistor_SMD:R_0402_1005Metric" V 6980 1750 50  0001 C CNN
@@
 	7050 3600 7050 5550
 $Comp
-L Connector_Generic:Conn_01x02 J?
+L Connector_Generic:Conn_01x02 J1
 U 1 1 5FADED1F
 P 1900 1550
-F 0 "J?" H 1818 1225 50  0000 C CNN
+F 0 "J1" H 1818 1225 50  0000 C CNN
 F 1 "Conn_01x02" H 1818 1316 50  0000 C CNN
-F 2 "" H 1900 1550 50  0001 C CNN
+F 2 "Connector_PinHeader_2.54mm:PinHeader_1x02_P2.54mm_Vertical" H 1900 1550 50  0001 C CNN
 F 3 "~" H 1900 1550 50  0001 C CNN
 	1    1900 1550
@@
 	2300 1550 2300 1650
 $Comp
-L B.B-eagle-import:VCC #V?
+L B.B-eagle-import:VCC #V07
 U 1 1 5FAF85B0
 P 7400 3050
-F 0 "#V?" H 7400 3050 50  0001 C CNN
+F 0 "#V07" H 7400 3050 50  0001 C CNN
 F 1 "VCC" H 7400 3180 59  0000 C CNN
 F 2 "" H 7400 3050 50  0001 C CNN
@@
 P 4500 2250
 AR Path="/5F77B818/5FB556D1" Ref="R?"  Part="1"
-AR Path="/5FB556D1" Ref="R?"  Part="1"
-F 0 "R?" H 4570 2296 50  0000 L CNN
+AR Path="/5FB556D1" Ref="R3"  Part="1"
+F 0 "R3" H 4570 2296 50  0000 L CNN
 F 1 "1M" H 4570 2205 50  0000 L CNN
 F 2 "Resistor_SMD:R_0402_1005Metric" V 4430 2250 50  0001 C CNN

Commit message: orezavani
smazaní A9G, SD karty, a zvuku
Parts:
- removed J1: Conn_01x02, Connector_PinHeader_2.54mm:PinHeader_1x02_P2.54mm_Vertical, symbol Connector_Generic:Conn_01x02
- removed J2, J3: Conn_01x08, Connector_PinHeader_2.54mm:PinHeader_1x08_P2.54mm_Vertical, symbol Connector_Generic:Conn_01x08
- added J? (x2): Conn_01x10, symbol Connector_Generic:Conn_01x10
- added J?: Conn_01x03, symbol Connector_Generic:Conn_01x03
- added Q?: SI3447CDV, BB:TSOP-6_1.5x3.0x0.95P, symbol B.B-rescue:Q_PMOS_DSG
- added R?: 100k, Resistor_SMD:R_0402_1005Metric, symbol Device:R
- R4: value 330k -> 300k; LCSC C25778 -> C25774
Connections:
- net labels added: bateri_temperatur
- net labels removed: SHUTDOWN_3V3, SHUTDOWN_5V
- wire segments 95 -> 97
Other:
- moved on the sheet: R1, R2, R3, R4

Commit message: nabijecka
Parts:
- removed J?: Conn_01x03, symbol Connector_Generic:Conn_01x03
- added J?: Conn_01x02, symbol Connector_Generic:Conn_01x02
- gave numbers to parts that had none: 4
Connections:
- net labels removed: bateri_temperatur
- wire segments 97 -> 101
Other:
- moved on the sheet: R3, R4

Commit message: odpojovan_nabijecky
Connections:
- net power00/VCC is gone; now on net charger00/BAT: Q4.1 (S), Q4.2, Q4.5, Q4.6
- net charger00/BAT: no longer J?.2 (Pin_2), Q4.4 (D)
- new net: J?.2 (Pin_2), Q4.4 (D)
Other:
- moved on the sheet: J2, J3, J?, Q4, R1, R2, R3, R4, R5

Commit message: 18650
Parts:
- removed J?: Conn_01x02, symbol Connector_Generic:Conn_01x02
- added BT1: Battery_Cell, BB:18650-holder, symbol B.B-rescue:Battery_Cell
- J2, J3: footprint (none) -> Connector_PinHeader_2.54mm:PinHeader_1x10_P2.54mm_Vertical
Connections:
- net at Q4.4 (D): now also BT1.1 (+), BT1.3 (+)
Changed lines of the file:
@@
 L B.B-eagle-import:GND #GND061
 U 1 1 5FA8F1DF
-P 2625 1800
-F 0 "#GND061" H 2625 1800 50  0001 C CNN
-F 1 "GND" H 2625 1720 59  0000 C CNN
-F 2 "" H 2625 1800 50  0001 C CNN
-F 3 "" H 2625 1800 50  0001 C CNN
-	1    2625 1800
+P 2275 2000
+F 0 "#GND061" H 2275 2000 50  0001 C CNN
+F 1 "GND" H 2275 1920 59  0000 C CNN
+F 2 "" H 2275 2000 50  0001 C CNN
+F 3 "" H 2275 2000 50  0001 C CNN
+	1    2275 2000
 	1    0    0    -1
 $EndComp
@@
 	7100 3250 7100 5050
 Wire Wire Line
-	2625 1600 2500 1600
-Wire Wire Line
-	2625 1600 2625 1700
+	2275 1850 2275 1900
 $Comp
 L B.B-eagle-import:VCC #V07
@@
 S 7500 1450 550  1300
 U 5FB26A97
-F0 "sheet5FB26A86" 50
+F0 "perception00" 50
 F1 "perception.sch" 50
 F2 "3V3" I L 7500 1600 50
@@
 F 0 "J2" V 7600 5700 50  0000 L CNN
 F 1 "Conn_01x10" V 7700 4700 50  0000 L CNN
-F 2 "" H 7600 5250 50  0001 C CNN
+F 2 "Connector_PinHeader_2.54mm:PinHeader_1x10_P2.54mm_Vertical" H 7600 5250 50  0001 C CNN
 F 3 "~" H 7600 5250 50  0001 C CNN
 	1    7600 5250
@@
 F 0 "J3" V 7800 5750 50  0000 C CNN
 F 1 "Conn_01x10" V 7900 4925 50  0000 C CNN
-F 2 "" H 7800 5250 50  0001 C CNN
+F 2 "Connector_PinHeader_2.54mm:PinHeader_1x10_P2.54mm_Vertical" H 7800 5250 50  0001 C CNN
 F 3 "~" H 7800 5250 50  0001 C CNN
 	1    7800 5250
@@
 $EndSheet
 $Comp
-L Connector_Generic:Conn_01x02 J?
-U 1 1 5FB6368C
-P 2300 1600
-F 0 "J?" H 2218 1275 50  0000 C CNN
-F 1 "Conn_01x02" H 2218 1366 50  0000 C CNN
-F 2 "" H 2300 1600 50  0001 C CNN
-F 3 "~" H 2300 1600 50  0001 C CNN
-	1    2300 1600
-	-1   0    0    1
-$EndComp
-$Comp
 L B.B-eagle-import:VCC #V06
 U 1 1 5FA8BF43
@@
 	5175 3000 5250 3000
 Wire Wire Line
-	2500 1500 2750 1500
+	2275 1500 2750 1500
 Wire Wire Line
 	3450 2700 3250 2700
 Wire Wire Line
 	3250 2700 3250 1500
+Wire Wire Line
+	2275 1550 2275 1500
+$Comp
+L B.B-rescue:Battery_Cell BT1
+U 1 1 5FBA1DA4
+P 2275 1750
+F 0 "BT1" H 2393 1846 50  0000 L CNN
+F 1 "Battery_Cell" H 2393 1755 50  0000 L CNN
+F 2 "BB:18650-holder" V 2275 1810 50  0001 C CNN
+F 3 "~" V 2275 1810 50  0001 C CNN
+	1    2275 1750
+	1    0    0    -1
+$EndComp
+$Comp
+L B.B-eagle-import:GND #GND0157
+U 1 1 5FBA25D8
+P 2075 2000
+F 0 "#GND0157" H 2075 2000 50  0001 C CNN
+F 1 "GND" H 2075 1920 59  0000 C CNN
+F 2 "" H 2075 2000 50  0001 C CNN
+F 3 "" H 2075 2000 50  0001 C CNN
+	1    2075 2000
+	1    0    0    -1
+$EndComp
+Wire Wire Line
+	2075 1850 2075 1900
+Wire Wire Line
+	2075 1550 2075 1500
+Wire Wire Line
+	2075 1500 2275 1500
+Connection ~ 2275 1500
 $EndSCHEMATC
