File: main_board/B.B/B.B.sch (KiCad schematic (older format))
At the start: 8 parts, among them J2 Conn_01x11, J3 Conn_01x11, Q11 SI3447CDV

Commit message: napajeni_na_stejne_strane
-poradi na konektoru
-napajeni IR prijmece z 5V na VCC
-vyssi nabijeci proud
-WS2812_power na IO21
Connections:
- net labels added: BAT+
- wire segments 103 -> 98

Commit message: uvolneni enkoderu
- dolomitelny enkoder
- zmenseni via u civek LDC
- vymena pouzdra USB-C
- otoceni IR prijmace
- zakas vylivani medi pod BMX9555
- odstraneni "ochrannych" odporu k M41T62
Changed lines of the file:
@@
 F10 "IO22" I R 6250 1800 50
 F11 "IO21" I R 6250 3750 50
-F12 "IO19" I R 6250 5350 50
-F13 "IO18" I R 6250 5250 50
+F12 "IO19" I R 6250 5250 50
+F13 "IO18" I R 6250 5350 50
 F14 "3V3" I L 5250 1700 50
 F15 "IO0-up" I R 6250 5450 50

Commit message: popisky
-popisky
-poladeni uddeleni enkoderu
-poladeni nayvu drah
-priopjeni gnd USB
-poligon V5 na led-desce do spodni vrstvu
Parts:
- F1, F2: symbol Device:Polyfuse -> B.B-rescue:Polyfuse-Device
- J2, J3: symbol Connector_Generic:Conn_01x11 -> B.B-rescue:Conn_01x11-Connector_Generic
- R1, R2: symbol Device:R -> B.B-rescue:R-Device
Changed lines of the file:
@@
 EESchema Schematic File Version 4
-LIBS:B.B-cache
-EELAYER 29 0
+EELAYER 30 0
 EELAYER END
 $Descr A4 11693 8268
@@
 	4300 2150 5250 2150
 $Comp
-L Device:R R?
+L B.B-rescue:R-Device R?
 U 1 1 5FA57DCC
 P 6900 1600
@@
 Wire Wire Line
 	8650 4450 8650 4700
-$Sheet
-S 3450 2625 850  175
-U 5FB8FF0F
-F0 "charger00" 50
-F1 "charger.sch" 50
-F2 "VCC" I R 4300 2700 50
-F3 "BAT" I L 3450 2700 50
-$EndSheet
 Wire Wire Line
 	4300 2700 5250 2700
@@
 	5000 3750 5250 3750
 $Comp
-L Connector_Generic:Conn_01x11 J2
+L B.B-rescue:Conn_01x11-Connector_Generic J2
 U 1 1 5FC8A4A2
 P 7600 5350
@@
 $EndComp
 $Comp
-L Device:Polyfuse F2
+L B.B-rescue:Polyfuse-Device F2
 U 1 1 5FC5EA4C
 P 2050 1700
@@
 $EndComp
 $Comp
-L Device:Polyfuse F1
+L B.B-rescue:Polyfuse-Device F1
 U 1 1 5FC5F6AE
 P 1850 1700
@@
 $EndSheet
 $Comp
-L Connector_Generic:Conn_01x11 J3
+L B.B-rescue:Conn_01x11-Connector_Generic J3
 U 1 1 5FC91920
 P 7800 5350
@@
 BAT+
 $Comp
-L Device:R R?
+L B.B-rescue:R-Device R?
 U 1 1 5FA54DFA
 P 6550 1600
@@
 Wire Wire Line
 	7175 1250 7175 3150
+$Sheet
+S 3450 2625 850  175
+U 5FB8FF0F
+F0 "charger00" 50
+F1 "charger.sch" 50
+F2 "VCC" I L 3450 2700 50
+F3 "BAT" I R 4300 2700 50
+$EndSheet
 $EndSCHEMATC

Commit message: LDC footprint
prodlouzeni pedu pro usnadneni rucniho osazovani
Parts:
- BT1: symbol B.B-rescue:Battery_Cell -> B.B-rescue:Battery_Cell-B.B-rescue
- F1, F2: symbol B.B-rescue:Polyfuse-Device -> B.B-rescue:Polyfuse-Device-B.B-rescue
- J2, J3: symbol B.B-rescue:Conn_01x11-Connector_Generic -> B.B-rescue:Conn_01x11-Connector_Generic-B.B-rescue
- Q11: symbol B.B-rescue:Q_PMOS_DSG -> B.B-rescue:Q_PMOS_DSG-B.B-rescue
- R1, R2: symbol B.B-rescue:R-Device -> B.B-rescue:R-Device-B.B-rescue
Changed lines of the file:
@@
 	7100 1400 7100 1600
 $Comp
-L B.B-eagle-import:VCC #V01
+L B.B-rescue:VCC-B.B-eagle-import #V01
 U 1 1 5FA8B2FC
 P 3375 1150
@@
 	4500 1500 4300 1500
 $Comp
-L B.B-eagle-import:+5V #V05
+L B.B-rescue:+5V-B.B-eagle-import #V05
 U 1 1 5F970ABB
 P 7350 1150
@@
 $EndComp
 $Comp
-L B.B-eagle-import:+3V3 #V04
+L B.B-rescue:+3V3-B.B-eagle-import #V04
 U 1 1 5F9711C3
 P 6550 1150
@@
 	4300 2150 5250 2150
 $Comp
-L B.B-rescue:R-Device R?
+L B.B-rescue:R-Device-B.B-rescue R?
 U 1 1 5FA57DCC
 P 6900 1600
@@
 	4500 1250 4500 1500
 $Comp
-L B.B-eagle-import:+5V #V02
+L B.B-rescue:+5V-B.B-eagle-import #V02
 U 1 1 5F96BCF7
 P 4500 1150
@@
 	5000 3750 5250 3750
 $Comp
-L B.B-rescue:Conn_01x11-Connector_Generic J2
+L B.B-rescue:Conn_01x11-Connector_Generic-B.B-rescue J2
 U 1 1 5FC8A4A2
 P 7600 5350
@@
 	3375 1700 3375 2700
 $Comp
-L B.B-eagle-import:GND #GND0156
+L B.B-rescue:GND-B.B-eagle-import #GND0156
 U 1 1 5FBE0F0B
 P 2725 1900
@@
 	1850 1550 1850 1500
 $Comp
-L B.B-eagle-import:GND #GND0157
+L B.B-rescue:GND-B.B-eagle-import #GND0157
 U 1 1 5FBA25D8
 P 1850 2250
@@
 $EndComp
 $Comp
-L B.B-rescue:Battery_Cell BT1
+L B.B-rescue:Battery_Cell-B.B-rescue BT1
 U 1 1 5FBA1DA4
 P 2050 2050
@@
 $EndComp
 $Comp
-L B.B-eagle-import:GND #GND061
+L B.B-rescue:GND-B.B-eagle-import #GND061
 U 1 1 5FA8F1DF
 P 2050 2250
@@
 	4800 1700 5250 1700
 $Comp
-L B.B-eagle-import:+3V3 #V03
+L B.B-rescue:+3V3-B.B-eagle-import #V03
 U 1 1 5F96C236
 P 4800 1150
@@
 	4800 1250 4800 1700
 $Comp
-L B.B-rescue:Q_PMOS_DSG Q?
+L B.B-rescue:Q_PMOS_DSG-B.B-rescue Q?
 U 1 1 5FBDC479
 P 2725 1600
@@
 $EndComp
 $Comp
-L B.B-rescue:Polyfuse-Device F2
+L B.B-rescue:Polyfuse-Device-B.B-rescue F2
 U 1 1 5FC5EA4C
 P 2050 1700
@@
 $EndComp
 $Comp
-L B.B-rescue:Polyfuse-Device F1
+L B.B-rescue:Polyfuse-Device-B.B-rescue F1
 U 1 1 5FC5F6AE
 P 1850 1700
@@
 $EndSheet
 $Comp
-L B.B-rescue:Conn_01x11-Connector_Generic J3
+L B.B-rescue:Conn_01x11-Connector_Generic-B.B-rescue J3
 U 1 1 5FC91920
 P 7800 5350
@@
 	7400 5450 6250 5450
 $Comp
-L B.B-eagle-import:GND #GND01
+L B.B-rescue:GND-B.B-eagle-import #GND01
 U 1 1 5FC953CE
 P 7325 6050
@@
 BAT+
 $Comp
-L B.B-rescue:R-Device R?
+L B.B-rescue:R-Device-B.B-rescue R?
 U 1 1 5FA54DFA
 P 6550 1600
@@
 	7500 3150 7175 3150
 $Comp
-L B.B-eagle-import:VCC #V07
+L B.B-rescue:VCC-B.B-eagle-import #V07
 U 1 1 5FAF85B0
 P 7175 1150

Commit message: JLCdata
- korekce pozice a natoceni
- data pro vyrobu
Parts:
- Q11: LCSC C145421 -> C144884
Connections:
- net labels added: +3.3V
- net labels removed: +3V3

Commit message: lucerna
Connections:
- net expanz00/5V-WS2812 is gone; now on net +5V: J2.10 (Pin_10), J2.11 (Pin_11)
- net ESP3200/IO0-up: no longer J2.5 (Pin_5)
Other:
- note added: "RB3203-Black_Box"
- note added: "Released under the Creative Commons Attribution-ShareAlike 4.0 License\nhttps://creativecommons.org/licenses/by-sa/4.0/\nDesigned by: Tom Vavrinec & RobotikaBrno\n\nRB3203-Black_Box\nhttps://github.com/XY"
- note added: "RoboticsBrno.eu\nRobotikaBrno.cz\nRobotarna"
- note added: "V1.1"
- moved on the sheet: BT1, F1, F2, J2, J3, Q11, R1, R2

Commit message: presuny_konektoru
Other:
- moved on the sheet: J2, J3
