File: main_board/B.B/perception.sch (KiCad schematic (older format))
At the start: 12 parts, among them U69 BMX055, U70 M41T62, U71 SPL06, Y1 32.768kHz

Commit message: nabijecka
Changed lines of the file:
@@
 $Descr A4 11693 8268
 encoding utf-8
-Sheet 5 7
+Sheet 5 8
 Title ""
 Date ""
@@
 AR Path="/5FA9DBB3/5F9F24D4/5F9701D7" Ref="U?"  Part="1"
 AR Path="/5F9EE529/5FB1300F/5F9701D7" Ref="U?"  Part="1"
-AR Path="/5FB26A97/5F9701D7" Ref="U?"  Part="1"
-F 0 "U?" H 6200 1875 50  0000 C CNN
+AR Path="/5FB26A97/5F9701D7" Ref="U61"  Part="1"
+F 0 "U61" H 6200 1875 50  0000 C CNN
 F 1 "BMX055" H 6200 1784 50  0000 C CNN
 F 2 "BB:LGA_4.5x3" H 5950 1650 50  0001 C CNN
@@
 AR Path="/5FA9DBB3/5F9F24D4/5F971B50" Ref="C?"  Part="1"
 AR Path="/5F9EE529/5FB1300F/5F971B50" Ref="C?"  Part="1"
-AR Path="/5FB26A97/5F971B50" Ref="C?"  Part="1"
-F 0 "C?" H 4665 1996 50  0000 L CNN
+AR Path="/5FB26A97/5F971B50" Ref="C67"  Part="1"
+F 0 "C67" H 4665 1996 50  0000 L CNN
 F 1 "10uf" H 4665 1905 50  0000 L CNN
 F 2 "Resistor_SMD:R_0805_2012Metric" H 4588 1800 50  0001 C CNN
@@
 AR Path="/5FA9DBB3/5F9F24D4/5F972192" Ref="#GND?"  Part="1"
 AR Path="/5F9EE529/5FB1300F/5F972192" Ref="#GND?"  Part="1"
-AR Path="/5FB26A97/5F972192" Ref="#GND?"  Part="1"
-F 0 "#GND?" H 4550 2200 50  0001 C CNN
+AR Path="/5FB26A97/5F972192" Ref="#GND0141"  Part="1"
+F 0 "#GND0141" H 4550 2200 50  0001 C CNN
 F 1 "GND" H 4550 2120 59  0000 C CNN
 F 2 "" H 4550 2200 50  0001 C CNN
@@
 AR Path="/5FA9DBB3/5F9F24D4/5F974417" Ref="C?"  Part="1"
 AR Path="/5F9EE529/5FB1300F/5F974417" Ref="C?"  Part="1"
-AR Path="/5FB26A97/5F974417" Ref="C?"  Part="1"
-F 0 "C?" H 5065 1996 50  0000 L CNN
+AR Path="/5FB26A97/5F974417" Ref="C68"  Part="1"
+F 0 "C68" H 5065 1996 50  0000 L CNN
 F 1 "0.1uf" H 5065 1905 50  0000 L CNN
 F 2 "Resistor_SMD:R_0805_2012Metric" H 4988 1800 50  0001 C CNN
@@
 AR Path="/5FA9DBB3/5F9F24D4/5F97A11B" Ref="#GND?"  Part="1"
 AR Path="/5F9EE529/5FB1300F/5F97A11B" Ref="#GND?"  Part="1"
-AR Path="/5FB26A97/5F97A11B" Ref="#GND?"  Part="1"
-F 0 "#GND?" H 4950 2200 50  0001 C CNN
+AR Path="/5FB26A97/5F97A11B" Ref="#GND0142"  Part="1"
+F 0 "#GND0142" H 4950 2200 50  0001 C CNN
 F 1 "GND" H 4950 2120 59  0000 C CNN
 F 2 "" H 4950 2200 50  0001 C CNN
@@
 AR Path="/5FA9DBB3/5F9F24D4/5F97F861" Ref="#GND?"  Part="1"
 AR Path="/5F9EE529/5FB1300F/5F97F861" Ref="#GND?"  Part="1"
-AR Path="/5FB26A97/5F97F861" Ref="#GND?"  Part="1"
-F 0 "#GND?" H 6100 2900 50  0001 C CNN
+AR Path="/5FB26A97/5F97F861" Ref="#GND0143"  Part="1"
+F 0 "#GND0143" H 6100 2900 50  0001 C CNN
 F 1 "GND" H 6100 2820 59  0000 C CNN
 F 2 "" H 6100 2900 50  0001 C CNN
@@
 AR Path="/5FA9DBB3/5F9F24D4/5F935E15" Ref="U?"  Part="1"
 AR Path="/5F9EE529/5FB1300F/5F935E15" Ref="U?"  Part="1"
-AR Path="/5FB26A97/5F935E15" Ref="U?"  Part="1"
-F 0 "U?" H 6125 3825 50  0000 C CNN
+AR Path="/5FB26A97/5F935E15" Ref="U67"  Part="1"
+F 0 "U67" H 6125 3825 50  0000 C CNN
 F 1 "M41T62" H 6125 3734 50  0000 C CNN
 F 2 "Package_DFN_QFN:QFN-16-1EP_3x3mm_P0.5mm_EP1.7x1.7mm" H 6100 3600 50  0001 C CNN
@@
 AR Path="/5FA9DBB3/5F9F24D4/5F93AF19" Ref="D?"  Part="1"
 AR Path="/5F9EE529/5FB1300F/5F93AF19" Ref="D?"  Part="1"
-AR Path="/5FB26A97/5F93AF19" Ref="D?"  Part="1"
-F 0 "D?" V 4746 3520 50  0000 R CNN
+AR Path="/5FB26A97/5F93AF19" Ref="D4"  Part="1"
+F 0 "D4" V 4746 3520 50  0000 R CNN
 F 1 "D" V 4655 3520 50  0000 R CNN
 F 2 "BB:SOD-323" H 4700 3600 50  0001 C CNN
@@
 AR Path="/5FA9DBB3/5F9F24D4/5F93D78D" Ref="Y?"  Part="1"
 AR Path="/5F9EE529/5FB1300F/5F93D78D" Ref="Y?"  Part="1"
-AR Path="/5FB26A97/5F93D78D" Ref="Y?"  Part="1"
-F 0 "Y?" V 6704 4231 50  0000 L CNN
+AR Path="/5FB26A97/5F93D78D" Ref="Y1"  Part="1"
+F 0 "Y1" V 6704 4231 50  0000 L CNN
 F 1 "32.768kHz" V 6795 4231 50  0000 L CNN
 F 2 "BB:SMD-3215_2P" H 6750 4100 50  0001 C CNN
@@
 AR Path="/5FA9DBB3/5F9F24D4/5F9470EF" Ref="#GND?"  Part="1"
 AR Path="/5F9EE529/5FB1300F/5F9470EF" Ref="#GND?"  Part="1"
-AR Path="/5FB26A97/5F9470EF" Ref="#GND?"  Part="1"
-F 0 "#GND?" H 6100 4250 50  0001 C CNN
+AR Path="/5FB26A97/5F9470EF" Ref="#GND0144"  Part="1"
+F 0 "#GND0144" H 6100 4250 50  0001 C CNN
 F 1 "GND" H 6100 4170 59  0000 C CNN
 F 2 "" H 6100 4250 50  0001 C CNN
@@
 AR Path="/5FA9DBB3/5F9F24D4/5F94A059" Ref="#GND?"  Part="1"
 AR Path="/5F9EE529/5FB1300F/5F94A059" Ref="#GND?"  Part="1"
-AR Path="/5FB26A97/5F94A059" Ref="#GND?"  Part="1"
-F 0 "#GND?" H 4950 4050 50  0001 C CNN
+AR Path="/5FB26A97/5F94A059" Ref="#GND0145"  Part="1"
+F 0 "#GND0145" H 4950 4050 50  0001 C CNN
 F 1 "GND" H 4950 3970 59  0000 C CNN
 F 2 "" H 4950 4050 50  0001 C CNN
@@
 AR Path="/5FA9DBB3/5F9F24D4/5F959D3B" Ref="#NC?"  Part="1"
 AR Path="/5F9EE529/5FB1300F/5F959D3B" Ref="#NC?"  Part="1"
-AR Path="/5FB26A97/5F959D3B" Ref="#NC?"  Part="1"
-F 0 "#NC?" H 6550 3600 50  0001 C CNN
+AR Path="/5FB26A97/5F959D3B" Ref="#NC26"  Part="1"
+F 0 "#NC26" H 6550 3600 50  0001 C CNN
 F 1 "NC" H 6550 3600 50  0001 C CNN
 F 2 "" H 6550 3600 50  0001 C CNN
@@
 AR Path="/5FA9DBB3/5F9F24D4/5F967811" Ref="U?"  Part="1"
 AR Path="/5F9EE529/5FB1300F/5F967811" Ref="U?"  Part="1"
-AR Path="/5FB26A97/5F967811" Ref="U?"  Part="1"
-F 0 "U?" H 6100 5225 50  0000 C CNN
+AR Path="/5FB26A97/5F967811" Ref="U69"  Part="1"
+F 0 "U69" H 6100 5225 50  0000 C CNN
 F 1 "SPL06" H 6100 5134 50  0000 C CNN
 F 2 "BB:SMD-8_2x2.5x0.65P" H 6100 5000 50  0001 C CNN
@@
 AR Path="/5FA9DBB3/5F9F24D4/5F96E1FD" Ref="#NC?"  Part="1"
 AR Path="/5F9EE529/5FB1300F/5F96E1FD" Ref="#NC?"  Part="1"
-AR Path="/5FB26A97/5F96E1FD" Ref="#NC?"  Part="1"
-F 0 "#NC?" H 6500 5300 50  0001 C CNN
+AR Path="/5FB26A97/5F96E1FD" Ref="#NC27"  Part="1"
+F 0 "#NC27" H 6500 5300 50  0001 C CNN
 F 1 "NC" H 6500 5300 50  0001 C CNN
 F 2 "" H 6500 5300 50  0001 C CNN
@@
 AR Path="/5FA9DBB3/5F9F24D4/5F970396" Ref="#NC?"  Part="1"
 AR Path="/5F9EE529/5FB1300F/5F970396" Ref="#NC?"  Part="1"
-AR Path="/5FB26A97/5F970396" Ref="#NC?"  Part="1"
-F 0 "#NC?" H 6850 2550 50  0001 C CNN
+AR Path="/5FB26A97/5F970396" Ref="#NC12"  Part="1"
+F 0 "#NC12" H 6850 2550 50  0001 C CNN
 F 1 "NC" H 6850 2550 50  0001 C CNN
 F 2 "" H 6850 2550 50  0001 C CNN
@@
 AR Path="/5FA9DBB3/5F9F24D4/5F970862" Ref="#NC?"  Part="1"
 AR Path="/5F9EE529/5FB1300F/5F970862" Ref="#NC?"  Part="1"
-AR Path="/5FB26A97/5F970862" Ref="#NC?"  Part="1"
-F 0 "#NC?" H 6850 2650 50  0001 C CNN
+AR Path="/5FB26A97/5F970862" Ref="#NC25"  Part="1"
+F 0 "#NC25" H 6850 2650 50  0001 C CNN
 F 1 "NC" H 6850 2650 50  0001 C CNN
 F 2 "" H 6850 2650 50  0001 C CNN
@@
 AR Path="/5FA9DBB3/5F9F24D4/5F970C9C" Ref="#NC?"  Part="1"
 AR Path="/5F9EE529/5FB1300F/5F970C9C" Ref="#NC?"  Part="1"
-AR Path="/5FB26A97/5F970C9C" Ref="#NC?"  Part="1"
-F 0 "#NC?" H 5550 2650 50  0001 C CNN
+AR Path="/5FB26A97/5F970C9C" Ref="#NC13"  Part="1"
+F 0 "#NC13" H 5550 2650 50  0001 C CNN
 F 1 "NC" H 5550 2650 50  0001 C CNN
 F 2 "" H 5550 2650 50  0001 C CNN
@@
 AR Path="/5FA9DBB3/5F9F24D4/5F975C33" Ref="C?"  Part="1"
 AR Path="/5F9EE529/5FB1300F/5F975C33" Ref="C?"  Part="1"
-AR Path="/5FB26A97/5F975C33" Ref="C?"  Part="1"
-F 0 "C?" H 5115 5246 50  0000 L CNN
+AR Path="/5FB26A97/5F975C33" Ref="C70"  Part="1"
+F 0 "C70" H 5115 5246 50  0000 L CNN
 F 1 "1uf" H 5115 5155 50  0000 L CNN
 F 2 "Resistor_SMD:R_0402_1005Metric" H 5038 5050 50  0001 C CNN
@@
 AR Path="/5FA9DBB3/5F9F24D4/5F975C39" Ref="#GND?"  Part="1"
 AR Path="/5F9EE529/5FB1300F/5F975C39" Ref="#GND?"  Part="1"
-AR Path="/5FB26A97/5F975C39" Ref="#GND?"  Part="1"
-F 0 "#GND?" H 5000 5450 50  0001 C CNN
+AR Path="/5FB26A97/5F975C39" Ref="#GND0146"  Part="1"
+F 0 "#GND0146" H 5000 5450 50  0001 C CNN
 F 1 "GND" H 5000 5370 59  0000 C CNN
 F 2 "" H 5000 5450 50  0001 C CNN
@@
 AR Path="/5FA9DBB3/5F9F24D4/5F9780C8" Ref="C?"  Part="1"
 AR Path="/5F9EE529/5FB1300F/5F9780C8" Ref="C?"  Part="1"
-AR Path="/5FB26A97/5F9780C8" Ref="C?"  Part="1"
-F 0 "C?" H 5065 3846 50  0000 L CNN
+AR Path="/5FB26A97/5F9780C8" Ref="C69"  Part="1"
+F 0 "C69" H 5065 3846 50  0000 L CNN
 F 1 "1uf" H 5065 3755 50  0000 L CNN
 F 2 "Resistor_SMD:R_0402_1005Metric" H 4988 3650 50  0001 C CNN
@@
 AR Path="/5FA9DBB3/5F9F24D4/5F98C0A7" Ref="#GND?"  Part="1"
 AR Path="/5F9EE529/5FB1300F/5F98C0A7" Ref="#GND?"  Part="1"
-AR Path="/5FB26A97/5F98C0A7" Ref="#GND?"  Part="1"
-F 0 "#GND?" H 6100 5650 50  0001 C CNN
+AR Path="/5FB26A97/5F98C0A7" Ref="#GND0147"  Part="1"
+F 0 "#GND0147" H 6100 5650 50  0001 C CNN
 F 1 "GND" H 6100 5570 59  0000 C CNN
 F 2 "" H 6100 5650 50  0001 C CNN
@@
 AR Path="/5FA9DBB3/5F9F24D4/5F990B4D" Ref="R?"  Part="1"
 AR Path="/5F9EE529/5FB1300F/5F990B4D" Ref="R?"  Part="1"
-AR Path="/5FB26A97/5F990B4D" Ref="R?"  Part="1"
-F 0 "R?" H 6920 5346 50  0000 L CNN
+AR Path="/5FB26A97/5F990B4D" Ref="R45"  Part="1"
+F 0 "R45" H 6920 5346 50  0000 L CNN
 F 1 "100k" H 6920 5255 50  0000 L CNN
 F 2 "Resistor_SMD:R_0402_1005Metric" V 6780 5300 50  0001 C CNN
@@
 AR Path="/5FA9DBB3/5F9F24D4/5F9924A7" Ref="#GND?"  Part="1"
 AR Path="/5F9EE529/5FB1300F/5F9924A7" Ref="#GND?"  Part="1"
-AR Path="/5FB26A97/5F9924A7" Ref="#GND?"  Part="1"
-F 0 "#GND?" H 6850 5550 50  0001 C CNN
+AR Path="/5FB26A97/5F9924A7" Ref="#GND0148"  Part="1"
+F 0 "#GND0148" H 6850 5550 50  0001 C CNN
 F 1 "GND" H 6850 5470 59  0000 C CNN
 F 2 "" H 6850 5550 50  0001 C CNN
@@
 AR Path="/5F9EE529/5F9F24D4/5FB01470" Ref="R46"  Part="1"
 AR Path="/5F9EE529/5FB1300F/5FB01470" Ref="R?"  Part="1"
-AR Path="/5FB26A97/5FB01470" Ref="R?"  Part="1"
-F 0 "R?" V 5450 4000 50  0000 C CNN
+AR Path="/5FB26A97/5FB01470" Ref="R9"  Part="1"
+F 0 "R9" V 5450 4000 50  0000 C CNN
 F 1 "220" V 5450 3800 50  0000 C CNN
 F 2 "Resistor_SMD:R_0402_1005Metric" V 5480 3900 50  0001 C CNN
@@
 AR Path="/5F9EE529/5F9F24D4/5FB01477" Ref="R47"  Part="1"
 AR Path="/5F9EE529/5FB1300F/5FB01477" Ref="R?"  Part="1"
-AR Path="/5FB26A97/5FB01477" Ref="R?"  Part="1"
-F 0 "R?" V 5650 4100 50  0000 C CNN
+AR Path="/5FB26A97/5FB01477" Ref="R39"  Part="1"
+F 0 "R39" V 5650 4100 50  0000 C CNN
 F 1 "220" V 5650 3900 50  0000 C CNN
 F 2 "Resistor_SMD:R_0402_1005Metric" V 5480 4000 50  0001 C CNN
