File: main_board/B.B/ESP32.sch (KiCad schematic (older format))
At the start: 39 parts, among them J5 USB_C_Receptacle_USB2.0, Q3 AO3400A, SW1 SW_DIP_x01, SW2 SW_DIP_x01, SW4 SW_DIP_x02, U64 CP2102N-A01-GQFN28, U65 ESP32-WROVER

Commit message: 18650
Parts:
- removed C105: 0.1uf, Capacitor_SMD:C_0805_2012Metric, symbol Device:C
- SW4: footprint (none) -> BB:SW-SMD-4; LCSC (none) -> C319052
- gave numbers to parts that had none: 1
Changed lines of the file:
@@
-$EndComp
-$Comp
-L Device:C C105
-U 1 1 5F8B431F
-P 4500 2150
-F 0 "C105" H 4615 2196 50  0000 L CNN
-F 1 "0.1uf" H 4615 2105 50  0000 L CNN
-F 2 "Capacitor_SMD:C_0805_2012Metric" H 4538 2000 50  0001 C CNN
-F 3 "~" H 4500 2150 50  0001 C CNN
-F 4 "C14663" H 4500 2150 50  0001 C CNN "LCSC"
-	1    4500 2150
-	1    0    0    -1
 $EndComp
 $Comp
@@
 F 0 "SW4" H 3375 2317 50  0000 C CNN
 F 1 "SW_DIP_x02" H 3375 2226 50  0000 C CNN
-F 2 "" H 3375 1950 50  0001 C CNN
-F 3 "~" H 3375 1950 50  0001 C CNN
+F 2 "BB:SW-SMD-4" H 3375 1950 50  0001 C CNN
+F 3 "https://datasheet.lcsc.com/szlcsc/2002271742_XKB-Connectivity-DSHP02TS-S_C319052.pdf" H 3375 1950 50  0001 C CNN
+F 4 "C319052" H 3375 1950 50  0001 C CNN "LCSC"
 	1    3375 1950
 	1    0    0    -1
@@
 AR Path="/5FA3274C/5FB94C99" Ref="R?"  Part="1"
 AR Path="/5F9EE529/5FB94C99" Ref="R?"  Part="1"
-AR Path="/5F77B818/5FB94C99" Ref="R?"  Part="1"
-F 0 "R?" V 5943 1250 50  0000 C CNN
+AR Path="/5F77B818/5FB94C99" Ref="R49"  Part="1"
+F 0 "R49" V 5943 1250 50  0000 C CNN
 F 1 "220" V 6034 1250 50  0000 C CNN
 F 2 "Resistor_SMD:R_0402_1005Metric" V 6080 1250 50  0001 C CNN

Commit message: polifuse
-filtr k prijmaci IR
-merwni bterky -> za zapinani
-odstraneni odpojovani nabijecky + oprava napajeciho prouhu
-odstraneni prevodniku napeti k WS2812
Parts:
- added C105: 0.1uf, Capacitor_SMD:C_0805_2012Metric, symbol Device:C
- R31, R32: value 5k1 -> 5.1k
Changed lines of the file:
@@
 $Descr A4 11693 8268
 encoding utf-8
-Sheet 8 8
+Sheet 6 8
 Title ""
 Date ""
@@
 $EndComp
 $Comp
-L B.B-eagle-import:GND #GND0121
-U 1 1 5F7B200A
-P 1600 3550
-F 0 "#GND0121" H 1600 3550 50  0001 C CNN
-F 1 "GND" H 1600 3429 59  0000 C CNN
-F 2 "" H 1600 3550 50  0001 C CNN
-F 3 "" H 1600 3550 50  0001 C CNN
-	1    1600 3550
-	1    0    0    -1
-$EndComp
-$Comp
 L Device:R R31
 U 1 1 5F7A8F71
 P 2800 2450
 F 0 "R31" H 2870 2496 50  0000 L CNN
-F 1 "5k1" H 2870 2405 50  0000 L CNN
+F 1 "5.1k" H 2870 2405 50  0000 L CNN
 F 2 "Resistor_SMD:R_0402_1005Metric" V 2730 2450 50  0001 C CNN
 F 3 "~" H 2800 2450 50  0001 C CNN
@@
 P 3100 2450
 F 0 "R32" H 3170 2496 50  0000 L CNN
-F 1 "5k1" H 3170 2405 50  0000 L CNN
+F 1 "5.1k" H 3170 2405 50  0000 L CNN
 F 2 "Resistor_SMD:R_0402_1005Metric" V 3030 2450 50  0001 C CNN
 F 3 "~" H 3100 2450 50  0001 C CNN
@@
 L B.B-eagle-import:LED LED1
 U 1 1 5FAD0890
-P 6800 3750
-F 0 "LED1" H 6878 3753 59  0000 L CNN
-F 1 "RED" H 6878 3648 59  0000 L CNN
-F 2 "LED_SMD:LED_0603_1608Metric" H 6800 3750 50  0001 C CNN
-F 3 "" H 6800 3750 50  0001 C CNN
-F 4 "C2286" H 6800 3750 50  0001 C CNN "LCSC"
-	1    6800 3750
-	1    0    0    -1
+P 7000 3850
+F 0 "LED1" H 7078 3853 59  0000 L CNN
+F 1 "RED" H 7078 3748 59  0000 L CNN
+F 2 "LED_SMD:LED_0603_1608Metric" H 7000 3850 50  0001 C CNN
+F 3 "" H 7000 3850 50  0001 C CNN
+F 4 "C2286" H 7000 3850 50  0001 C CNN "LCSC"
+	1    7000 3850
+	-1   0    0    1
 $EndComp
 $Comp
 L B.B-eagle-import:LED LED2
 U 1 1 5FAD1734
-P 7250 3750
-F 0 "LED2" H 7328 3753 59  0000 L CNN
-F 1 "RED" H 7328 3648 59  0000 L CNN
-F 2 "LED_SMD:LED_0603_1608Metric" H 7250 3750 50  0001 C CNN
-F 3 "" H 7250 3750 50  0001 C CNN
-F 4 "C2286" H 7250 3750 50  0001 C CNN "LCSC"
-	1    7250 3750
-	1    0    0    -1
+P 7450 3850
+F 0 "LED2" H 7528 3853 59  0000 L CNN
+F 1 "RED" H 7528 3748 59  0000 L CNN
+F 2 "LED_SMD:LED_0603_1608Metric" H 7450 3850 50  0001 C CNN
+F 3 "" H 7450 3850 50  0001 C CNN
+F 4 "C2286" H 7450 3850 50  0001 C CNN "LCSC"
+	1    7450 3850
+	-1   0    0    1
 $EndComp
 $Comp
 L B.B-eagle-import:GND #GND0117
 U 1 1 5FAD557F
-P 7250 4050
-F 0 "#GND0117" H 7250 4050 50  0001 C CNN
-F 1 "GND" H 7250 3929 59  0000 C CNN
-F 2 "" H 7250 4050 50  0001 C CNN
-F 3 "" H 7250 4050 50  0001 C CNN
-	1    7250 4050
+P 7450 4050
+F 0 "#GND0117" H 7450 4050 50  0001 C CNN
+F 1 "GND" H 7450 3929 59  0000 C CNN
+F 2 "" H 7450 4050 50  0001 C CNN
+F 3 "" H 7450 4050 50  0001 C CNN
+	1    7450 4050
 	1    0    0    -1
 $EndComp
@@
 L B.B-eagle-import:GND #GND0116
 U 1 1 5FAD5963
-P 6800 4050
-F 0 "#GND0116" H 6800 4050 50  0001 C CNN
-F 1 "GND" H 6800 3929 59  0000 C CNN
-F 2 "" H 6800 4050 50  0001 C CNN
-F 3 "" H 6800 4050 50  0001 C CNN
-	1    6800 4050
-	1    0    0    -1
-$EndComp
-Wire Wire Line
-	6800 3350 6800 3250
+P 7000 4050
+F 0 "#GND0116" H 7000 4050 50  0001 C CNN
+F 1 "GND" H 7000 3929 59  0000 C CNN
+F 2 "" H 7000 4050 50  0001 C CNN
+F 3 "" H 7000 4050 50  0001 C CNN
+	1    7000 4050
+	1    0    0    -1
+$EndComp
+Wire Wire Line
+	7000 3350 7000 3250
 $Comp
 L Device:R R?
@@
 L Device:R R?
 U 1 1 5FA643BB
-P 7250 3500
+P 7450 3500
 AR Path="/5FA3274C/5FA643BB" Ref="R?"  Part="1"
 AR Path="/5F9EE529/5FA643BB" Ref="R?"  Part="1"
 AR Path="/5F77B818/5FA643BB" Ref="R27"  Part="1"
-F 0 "R27" V 7043 3500 50  0000 C CNN
-F 1 "220" V 7134 3500 50  0000 C CNN
-F 2 "Resistor_SMD:R_0402_1005Metric" V 7180 3500 50  0001 C CNN
-F 3 "~" H 7250 3500 50  0001 C CNN
-F 4 "C25092" V 7250 3500 50  0001 C CNN "LCSC"
-	1    7250 3500
+F 0 "R27" V 7625 3500 50  0000 C CNN
+F 1 "220" V 7550 3500 50  0000 C CNN
+F 2 "Resistor_SMD:R_0402_1005Metric" V 7380 3500 50  0001 C CNN
+F 3 "~" H 7450 3500 50  0001 C CNN
+F 4 "C25092" V 7450 3500 50  0001 C CNN "LCSC"
+	1    7450 3500
 	-1   0    0    1
 $EndComp
@@
 L Device:R R?
 U 1 1 5FA646C4
-P 6800 3500
+P 7000 3500
 AR Path="/5FA3274C/5FA646C4" Ref="R?"  Part="1"
 AR Path="/5F9EE529/5FA646C4" Ref="R?"  Part="1"
 AR Path="/5F77B818/5FA646C4" Ref="R26"  Part="1"
-F 0 "R26" V 6593 3500 50  0000 C CNN
-F 1 "220" V 6684 3500 50  0000 C CNN
-F 2 "Resistor_SMD:R_0402_1005Metric" V 6730 3500 50  0001 C CNN
-F 3 "~" H 6800 3500 50  0001 C CNN
-F 4 "C25092" V 6800 3500 50  0001 C CNN "LCSC"
-	1    6800 3500
+F 0 "R26" V 7175 3500 50  0000 C CNN
+F 1 "220" V 7100 3500 50  0000 C CNN
+F 2 "Resistor_SMD:R_0402_1005Metric" V 6930 3500 50  0001 C CNN
+F 3 "~" H 7000 3500 50  0001 C CNN
+F 4 "C25092" V 7000 3500 50  0001 C CNN "LCSC"
+	1    7000 3500
 	-1   0    0    1
 $EndComp
@@
 	6450 1850 6750 1850
 Wire Wire Line
-	6800 3250 6450 3250
-Wire Wire Line
-	6450 3150 7250 3150
-Wire Wire Line
-	7250 3150 7250 3350
+	7000 3250 6450 3250
+Wire Wire Line
+	6450 3150 7450 3150
+Wire Wire Line
+	7450 3150 7450 3350
 $Comp
 L B.B-rescue:Q_NPN_BCE MMBT3904
@@
 	6000 1250 5950 1250
 Connection ~ 5950 1250
+$Comp
+L Device:C C105
+U 1 1 5FBE5B3C
+P 4500 2150
+F 0 "C105" H 4615 2196 50  0000 L CNN
+F 1 "0.1uf" H 4615 2105 50  0000 L CNN
+F 2 "Capacitor_SMD:C_0805_2012Metric" H 4538 2000 50  0001 C CNN
+F 3 "~" H 4500 2150 50  0001 C CNN
+F 4 "C15850" H 4500 2150 50  0001 C CNN "LCSC"
+	1    4500 2150
+	1    0    0    -1
+$EndComp
+$Comp
+L B.B-eagle-import:NC #NC28
+U 1 1 5FC5D9A0
+P 1600 3450
+F 0 "#NC28" H 1600 3450 50  0001 C CNN
+F 1 "NC" H 1600 3450 50  0001 C CNN
+F 2 "" H 1600 3450 50  0001 C CNN
+F 3 "" H 1600 3450 50  0001 C CNN
+	1    1600 3450
+	0    1    1    0
+$EndComp
 $EndSCHEMATC

Commit message: lenky_k_CP2102
Connections:
- wire segments 103 -> 109
Changed lines of the file:
@@
 L B.B-eagle-import:LED LED1
 U 1 1 5FAD0890
-P 7000 3850
-F 0 "LED1" H 7078 3853 59  0000 L CNN
-F 1 "RED" H 7078 3748 59  0000 L CNN
-F 2 "LED_SMD:LED_0603_1608Metric" H 7000 3850 50  0001 C CNN
-F 3 "" H 7000 3850 50  0001 C CNN
-F 4 "C2286" H 7000 3850 50  0001 C CNN "LCSC"
-	1    7000 3850
-	-1   0    0    1
+P 7400 2575
+F 0 "LED1" H 7478 2578 59  0000 L CNN
+F 1 "RED" H 7478 2473 59  0000 L CNN
+F 2 "LED_SMD:LED_0603_1608Metric" H 7400 2575 50  0001 C CNN
+F 3 "" H 7400 2575 50  0001 C CNN
+F 4 "C2286" H 7400 2575 50  0001 C CNN "LCSC"
+	1    7400 2575
+	1    0    0    -1
 $EndComp
 $Comp
 L B.B-eagle-import:LED LED2
 U 1 1 5FAD1734
-P 7450 3850
-F 0 "LED2" H 7528 3853 59  0000 L CNN
-F 1 "RED" H 7528 3748 59  0000 L CNN
-F 2 "LED_SMD:LED_0603_1608Metric" H 7450 3850 50  0001 C CNN
-F 3 "" H 7450 3850 50  0001 C CNN
-F 4 "C2286" H 7450 3850 50  0001 C CNN "LCSC"
-	1    7450 3850
-	-1   0    0    1
-$EndComp
-$Comp
-L B.B-eagle-import:GND #GND0117
-U 1 1 5FAD557F
-P 7450 4050
-F 0 "#GND0117" H 7450 4050 50  0001 C CNN
-F 1 "GND" H 7450 3929 59  0000 C CNN
-F 2 "" H 7450 4050 50  0001 C CNN
-F 3 "" H 7450 4050 50  0001 C CNN
-	1    7450 4050
-	1    0    0    -1
-$EndComp
-$Comp
-L B.B-eagle-import:GND #GND0116
-U 1 1 5FAD5963
-P 7000 4050
-F 0 "#GND0116" H 7000 4050 50  0001 C CNN
-F 1 "GND" H 7000 3929 59  0000 C CNN
-F 2 "" H 7000 4050 50  0001 C CNN
-F 3 "" H 7000 4050 50  0001 C CNN
-	1    7000 4050
-	1    0    0    -1
-$EndComp
-Wire Wire Line
-	7000 3350 7000 3250
+P 6950 2575
+F 0 "LED2" H 7028 2578 59  0000 L CNN
+F 1 "RED" H 7028 2473 59  0000 L CNN
+F 2 "LED_SMD:LED_0603_1608Metric" H 6950 2575 50  0001 C CNN
+F 3 "" H 6950 2575 50  0001 C CNN
+F 4 "C2286" H 6950 2575 50  0001 C CNN "LCSC"
+	1    6950 2575
+	1    0    0    -1
+$EndComp
+Wire Wire Line
+	7400 3075 7400 3250
 $Comp
 L Device:R R?
@@
 L Device:R R?
 U 1 1 5FA643BB
-P 7450 3500
+P 6950 2925
 AR Path="/5FA3274C/5FA643BB" Ref="R?"  Part="1"
 AR Path="/5F9EE529/5FA643BB" Ref="R?"  Part="1"
 AR Path="/5F77B818/5FA643BB" Ref="R27"  Part="1"
-F 0 "R27" V 7625 3500 50  0000 C CNN
-F 1 "220" V 7550 3500 50  0000 C CNN
-F 2 "Resistor_SMD:R_0402_1005Metric" V 7380 3500 50  0001 C CNN
-F 3 "~" H 7450 3500 50  0001 C CNN
-F 4 "C25092" V 7450 3500 50  0001 C CNN "LCSC"
-	1    7450 3500
-	-1   0    0    1
+F 0 "R27" V 7125 2925 50  0000 C CNN
+F 1 "220" V 7050 2925 50  0000 C CNN
+F 2 "Resistor_SMD:R_0402_1005Metric" V 6880 2925 50  0001 C CNN
+F 3 "~" H 6950 2925 50  0001 C CNN
+F 4 "C25092" V 6950 2925 50  0001 C CNN "LCSC"
+	1    6950 2925
+	1    0    0    -1
 $EndComp
 $Comp
 L Device:R R?
 U 1 1 5FA646C4
-P 7000 3500
+P 7400 2925
 AR Path="/5FA3274C/5FA646C4" Ref="R?"  Part="1"
 AR Path="/5F9EE529/5FA646C4" Ref="R?"  Part="1"
 AR Path="/5F77B818/5FA646C4" Ref="R26"  Part="1"
-F 0 "R26" V 7175 3500 50  0000 C CNN
-F 1 "220" V 7100 3500 50  0000 C CNN
-F 2 "Resistor_SMD:R_0402_1005Metric" V 6930 3500 50  0001 C CNN
-F 3 "~" H 7000 3500 50  0001 C CNN
-F 4 "C25092" V 7000 3500 50  0001 C CNN "LCSC"
-	1    7000 3500
-	-1   0    0    1
+F 0 "R26" V 7575 2925 50  0000 C CNN
+F 1 "220" V 7500 2925 50  0000 C CNN
+F 2 "Resistor_SMD:R_0402_1005Metric" V 7330 2925 50  0001 C CNN
+F 3 "~" H 7400 2925 50  0001 C CNN
+F 4 "C25092" V 7400 2925 50  0001 C CNN "LCSC"
+	1    7400 2925
+	1    0    0    -1
 $EndComp
 Text HLabel 2800 1850 1    50   Input ~ 0
@@
 	6450 1850 6750 1850
 Wire Wire Line
-	7000 3250 6450 3250
-Wire Wire Line
-	6450 3150 7450 3150
-Wire Wire Line
-	7450 3150 7450 3350
+	7400 3250 6450 3250
+Wire Wire Line
+	6450 3150 6950 3150
+Wire Wire Line
+	6950 3150 6950 3075
 $Comp
 L B.B-rescue:Q_NPN_BCE MMBT3904
@@
 	0    1    1    0
 $EndComp
+Wire Wire Line
+	7400 2475 7400 2425
+Wire Wire Line
+	7400 2425 6950 2425
+Wire Wire Line
+	6950 2425 6950 2475
+Wire Wire Line
+	7400 2425 7400 950
+Wire Wire Line
+	5350 950  5350 1250
+Connection ~ 7400 2425
+Wire Wire Line
+	7400 950  5350 950
 $EndSCHEMATC

Commit message: uvolneni enkoderu
- dolomitelny enkoder
- zmenseni via u civek LDC
- vymena pouzdra USB-C
- otoceni IR prijmace
- zakas vylivani medi pod BMX9555
- odstraneni "ochrannych" odporu k M41T62
Parts:
- removed C105: 0.1uf, Capacitor_SMD:C_0805_2012Metric, symbol Device:C
- removed C106: 10uf, Capacitor_SMD:C_0805_2012Metric, symbol Device:C
- J5: footprint Connector_USB:USB_C_Receptacle_Amphenol_12401610E4-2A -> BB:USB_C_Female-16Pin-HPJF
Connections:
- wire segments 109 -> 107
Changed lines of the file:
@@
 F 0 "J5" H 2007 3417 50  0000 C CNN
 F 1 "USB_C_Receptacle_USB2.0" H 2007 3326 50  0000 C CNN
-F 2 "Connector_USB:USB_C_Receptacle_Amphenol_12401610E4-2A" H 2050 2550 50  0001 C CNN
+F 2 "BB:USB_C_Female-16Pin-HPJF" H 2050 2550 50  0001 C CNN
 F 3 "https://www.usb.org/sites/default/files/documents/usb_type-c.zip" H 2050 2550 50  0001 C CNN
 	1    1900 2550
@@
 Wire Wire Line
 	4500 1300 4500 1250
-$Comp
-L Device:C C106
-U 1 1 5F8B4312
-P 4950 2150
-F 0 "C106" H 5065 2196 50  0000 L CNN
-F 1 "10uf" H 5065 2105 50  0000 L CNN
-F 2 "Capacitor_SMD:C_0805_2012Metric" H 4988 2000 50  0001 C CNN
-F 3 "~" H 4950 2150 50  0001 C CNN
-F 4 "C15850" H 4950 2150 50  0001 C CNN "LCSC"
-	1    4950 2150
-	1    0    0    -1
-$EndComp
-$Comp
-L B.B-eagle-import:GND #GND0115
-U 1 1 5F8B4318
-P 4950 2400
-F 0 "#GND0115" H 4950 2400 50  0001 C CNN
-F 1 "GND" H 4950 2350 59  0000 C CNN
-F 2 "" H 4950 2400 50  0001 C CNN
-F 3 "" H 4950 2400 50  0001 C CNN
-	1    4950 2400
-	1    0    0    -1
-$EndComp
-$Comp
-L B.B-eagle-import:GND #GND0114
-U 1 1 5F8B4325
-P 4500 2400
-F 0 "#GND0114" H 4500 2400 50  0001 C CNN
-F 1 "GND" H 4500 2350 59  0000 C CNN
-F 2 "" H 4500 2400 50  0001 C CNN
-F 3 "" H 4500 2400 50  0001 C CNN
-	1    4500 2400
-	1    0    0    -1
-$EndComp
-Wire Wire Line
-	4950 2000 4950 1950
-Wire Wire Line
-	4500 2000 4500 1950
 Wire Wire Line
 	2750 5025 2750 4975
@@
 Connection ~ 4950 1250
 Wire Wire Line
-	4950 1250 5350 1250
-Connection ~ 4950 1950
-Wire Wire Line
-	4950 1950 5450 1950
+	4950 1250 5250 1250
 $Comp
 L Device:R R22
@@
 Wire Wire Line
 	4150 1250 4500 1250
-Connection ~ 4150 1950
-Connection ~ 4500 1950
-Wire Wire Line
-	4500 1950 4950 1950
 Wire Wire Line
 	3900 1950 4150 1950
-Wire Wire Line
-	4150 1950 4500 1950
 Text HLabel 6300 1250 2    50   Input ~ 0
 cable_connected
@@
 Connection ~ 5950 1250
 $Comp
-L Device:C C105
-U 1 1 5FBE5B3C
-P 4500 2150
-F 0 "C105" H 4615 2196 50  0000 L CNN
-F 1 "0.1uf" H 4615 2105 50  0000 L CNN
-F 2 "Capacitor_SMD:C_0805_2012Metric" H 4538 2000 50  0001 C CNN
-F 3 "~" H 4500 2150 50  0001 C CNN
-F 4 "C15850" H 4500 2150 50  0001 C CNN "LCSC"
-	1    4500 2150
-	1    0    0    -1
-$EndComp
-$Comp
 L B.B-eagle-import:NC #NC28
 U 1 1 5FC5D9A0
@@
 Wire Wire Line
 	7400 950  5350 950
+Wire Wire Line
+	5450 1950 5250 1950
+Wire Wire Line
+	5250 1950 5250 1250
+Connection ~ 5250 1250
+Wire Wire Line
+	5250 1250 5350 1250
 $EndSCHEMATC

Commit message: popisky
-popisky
-poladeni uddeleni enkoderu
-poladeni nayvu drah
-priopjeni gnd USB
-poligon V5 na led-desce do spodni vrstvu
Parts:
- C102, C103, C104, C107, C108, C109: symbol Device:C -> B.B-rescue:C-Device
- Q3: symbol Transistor_FET:2N7002 -> B.B-rescue:2N7002-Transistor_FET
- R20, R21, R22, R23, R24, R25, R26, R27, R28, R29, R30, R31, R32, R33, R34, R35, R36, R37, R38, R49: symbol Device:R -> B.B-rescue:R-Device
- SW1, SW2: symbol Switch:SW_DIP_x01 -> B.B-rescue:SW_DIP_x01-Switch
- SW4: symbol Switch:SW_DIP_x02 -> B.B-rescue:SW_DIP_x02-Switch
- U64: symbol Interface_USB:CP2102N-A01-GQFN28 -> B.B-rescue:CP2102N-A01-GQFN28-Interface_USB
Changed lines of the file:
@@
 EESchema Schematic File Version 4
-LIBS:B.B-cache
-EELAYER 29 0
+EELAYER 30 0
 EELAYER END
 $Descr A4 11693 8268
 encoding utf-8
-Sheet 4 8
+Sheet 3 8
 Title ""
 Date ""
@@
 $EndComp
 $Comp
-L Device:R R31
+L B.B-rescue:R-Device R31
 U 1 1 5F7A8F71
 P 2800 2450
@@
 Connection ~ 3450 5075
 $Comp
-L Device:R R33
+L B.B-rescue:R-Device R33
 U 1 1 5F80B567
 P 8900 3350
@@
 $EndComp
 $Comp
-L Device:R R37
+L B.B-rescue:R-Device R37
 U 1 1 5F82433D
 P 8900 3850
@@
 $EndComp
 $Comp
-L Device:R R35
+L B.B-rescue:R-Device R35
 U 1 1 5F8281DA
 P 8900 3600
@@
 	9150 3350 9150 3600
 $Comp
-L Device:C C103
+L B.B-rescue:C-Device C103
 U 1 1 5F84DAE6
 P 4950 1450
@@
 	4950 1300 4950 1250
 $Comp
-L Device:C C102
+L B.B-rescue:C-Device C102
 U 1 1 5F8566B5
 P 4500 1450
@@
 $EndComp
 $Comp
-L Device:C C109
+L B.B-rescue:C-Device C109
 U 1 1 5F970DFC
 P 2750 5175
@@
 $EndComp
 $Comp
-L Device:C C108
+L B.B-rescue:C-Device C108
 U 1 1 5F971517
 P 2300 5175
@@
 D-
 $Comp
-L Device:R R34
+L B.B-rescue:R-Device R34
 U 1 1 5F7BE1D0
 P 9800 3350
@@
 $EndComp
 $Comp
-L Device:R R36
+L B.B-rescue:R-Device R36
 U 1 1 5F7BE95B
 P 9800 3600
@@
 IO18
 $Comp
-L Transistor_FET:2N7002 Q3
+L B.B-rescue:2N7002-Transistor_FET Q3
 U 1 1 5F83FB30
 P 3900 1350
@@
 	3700 1250 3600 1250
 $Comp
-L Device:R R28
+L B.B-rescue:R-Device R28
 U 1 1 5F860400
 P 4150 2150
@@
 	2500 1950 2800 1950
 $Comp
-L Switch:SW_DIP_x01 SW1
+L B.B-rescue:SW_DIP_x01-Switch SW1
 U 1 1 5F90B5A3
 P 7650 5400
@@
 $EndComp
 $Comp
-L Device:R R20
+L B.B-rescue:R-Device R20
 U 1 1 5F913318
 P 8200 5400
@@
 Connection ~ 8000 5400
 $Comp
-L Device:R R30
+L B.B-rescue:R-Device R30
 U 1 1 5F936AC5
 P 9900 5400
@@
 EN
 $Comp
-L Device:R R21
+L B.B-rescue:R-Device R21
 U 1 1 5F898834
 P 4150 1450
@@
 $EndComp
 $Comp
-L Interface_USB:CP2102N-A01-GQFN28 U64
+L B.B-rescue:CP2102N-A01-GQFN28-Interface_USB U64
 U 1 1 5F78AFDC
 P 5950 2650
@@
 	4950 1250 5250 1250
 $Comp
-L Device:R R22
+L B.B-rescue:R-Device R22
 U 1 1 5F8D7784
 P 5350 1450
@@
 	8975 1800 9150 1800
 $Comp
-L Device:R R23
+L B.B-rescue:R-Device R23
 U 1 1 5F9B97DB
 P 9350 1800
@@
 $EndComp
 $Comp
-L Device:R R29
+L B.B-rescue:R-Device R29
 U 1 1 5F9BA036
 P 9350 2450
@@
 $EndComp
 $Comp
-L Device:C C104
+L B.B-rescue:C-Device C104
 U 1 1 5FABBE4E
 P 7650 5650
@@
 $EndComp
 $Comp
-L Device:R R32
+L B.B-rescue:R-Device R32
 U 1 1 5FAC0DBD
 P 3100 2450
@@
 	7400 3075 7400 3250
 $Comp
-L Device:R R?
+L B.B-rescue:R-Device R?
 U 1 1 5FA6121E
 P 6900 1750
@@
 $EndComp
 $Comp
-L Device:R R?
+L B.B-rescue:R-Device R?
 U 1 1 5FA64256
 P 6900 1850
@@
 $EndComp
 $Comp
-L Device:R R?
+L B.B-rescue:R-Device R?
 U 1 1 5FA643BB
 P 6950 2925
@@
 $EndComp
 $Comp
-L Device:R R?
+L B.B-rescue:R-Device R?
 U 1 1 5FA646C4
 P 7400 2925
@@
 	2800 1950 3075 1950
 $Comp
-L Switch:SW_DIP_x01 SW2
+L B.B-rescue:SW_DIP_x01-Switch SW2
 U 1 1 5FB1B20F
 P 9350 5400
@@
 $EndComp
 $Comp
-L Device:C C107
+L B.B-rescue:C-Device C107
 U 1 1 5FB1BF0E
 P 9350 5650
@@
 	10050 5400 10200 5400
 $Comp
-L Device:R R38
+L B.B-rescue:R-Device R38
 U 1 1 5FBD064E
 P 3450 4725
@@
 $EndComp
 $Comp
-L Switch:SW_DIP_x02 SW4
+L B.B-rescue:SW_DIP_x02-Switch SW4
 U 1 1 5FB55D9C
 P 3375 1950
@@
 cable_connected
 $Comp
-L Device:R R?
+L B.B-rescue:R-Device R?
 U 1 1 5FB94C99
 P 6150 1250

Commit message: LDC footprint
prodlouzeni pedu pro usnadneni rucniho osazovani
Parts:
- C102, C103, C104, C107, C108, C109: symbol B.B-rescue:C-Device -> B.B-rescue:C-Device-B.B-rescue
- J5: symbol B.B-rescue:USB_C_Receptacle_USB2.0-Connector -> B.B-rescue:USB_C_Receptacle_USB2.0-Connector-B.B-rescue
- LED1, LED2: symbol B.B-eagle-import:LED -> B.B-rescue:LED-B.B-eagle-import
- MMBT1, MMBT3904: symbol B.B-rescue:Q_NPN_BCE -> B.B-rescue:Q_NPN_BCE-B.B-rescue
- Q3: symbol B.B-rescue:2N7002-Transistor_FET -> B.B-rescue:2N7002-Transistor_FET-B.B-rescue
- R20, R21, R22, R23, R24, R25, R26, R27, R28, R29, R30, R31, R32, R33, R34, R35, R36, R37, R38, R49: symbol B.B-rescue:R-Device -> B.B-rescue:R-Device-B.B-rescue
- SW1, SW2: symbol B.B-rescue:SW_DIP_x01-Switch -> B.B-rescue:SW_DIP_x01-Switch-B.B-rescue
- SW4: symbol B.B-rescue:SW_DIP_x02-Switch -> B.B-rescue:SW_DIP_x02-Switch-B.B-rescue
- U64: symbol B.B-rescue:CP2102N-A01-GQFN28-Interface_USB -> B.B-rescue:CP2102N-A01-GQFN28-Interface_USB-B.B-rescue
- U65: symbol B.B-rescue:ESP32-WROVER-B.B-eagle-import -> B.B-rescue:ESP32-WROVER-B.B-eagle-import-B.B-rescue; LCSC (none) -> C503591
