File: main_board/B.B/ledDeska.kicad_pcb (KiCad board)
At the start: 2 copper layers, 94 x 94 mm, 134 parts, among them J3 Conn_01x11, U1 WS2812, U10 WS2812, U11 WS2812, U12 WS2812, U13 WS2812, U14 WS2812, U15 WS2812, U16 WS2812, U17 WS2812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

Commit message: JLCdata
- korekce pozice a natoceni
- data pro vyrobu
Parts:
- U66: footprint Package_DFN_QFN:WQFN-16-1EP_4x4mm_P0.5mm_EP2.6x2.6mm_ThermalVias -> BB:WQFN-16_4x4mm
Routing:
- net /next-board00/LDC-GND: track 37.6 -> 39.5 mm
Other:
- rule via_min_size: 0.4 -> 0.35
