File: main_board/B.B/charger.sch (KiCad schematic (older format))
At the start: 8 parts

Commit message: odpojovan_nabijecky
Parts:
- added Q?: SI3447CDV, BB:TSOP-6_1.5x3.0x0.95P, symbol B.B-rescue:Q_PMOS_DSG
- added Q?: 2N7002, Package_TO_SOT_SMD:SOT-23, symbol Transistor_FET:2N7002
- added R?: 1M, Resistor_SMD:R_0402_1005Metric, symbol Device:R
Connections:
- wire segments 17 -> 26
Changed lines of the file:
@@
 Wire Wire Line
 	4100 3250 4175 3250
-Text HLabel 7000 3250 2    50   Input ~ 0
+Text HLabel 8000 3250 2    50   Input ~ 0
 BAT
 $Comp
@@
 U 1 1 5FC03C27
 P 5250 3400
-F 0 "R?" V 5325 3375 50  0000 R CNN
-F 1 "1,2k" V 5325 3550 50  0000 R CNN
+F 0 "R?" V 5300 3275 50  0000 R CNN
+F 1 "1,2k" V 5325 3500 50  0000 R CNN
 F 2 "Resistor_SMD:R_0402_1005Metric" V 5180 3400 50  0001 C CNN
 F 3 "~" H 5250 3400 50  0001 C CNN
@@
 U 1 1 5FC04CCC
 P 5250 3625
-F 0 "R?" V 5325 3750 50  0000 R CNN
-F 1 "1,2k" V 5325 3650 50  0000 R CNN
+F 0 "R?" V 5325 3850 50  0000 R CNN
+F 1 "1,2k" V 5175 3700 50  0000 R CNN
 F 2 "Resistor_SMD:R_0402_1005Metric" V 5180 3625 50  0001 C CNN
 F 3 "~" H 5250 3625 50  0001 C CNN
@@
 Connection ~ 6875 3250
 Wire Wire Line
-	6875 3250 7000 3250
+	6875 3250 7350 3250
 $Comp
 L B.B-rescue:SE9017 U?
@@
 Wire Wire Line
 	4175 3250 4750 3250
+$Comp
+L B.B-rescue:Q_PMOS_DSG Q?
+U 1 1 5FBB8789
+P 7550 3350
+AR Path="/5F9EE529/5FBB8789" Ref="Q?"  Part="1"
+AR Path="/5FA4C94D/5FBB8789" Ref="Q?"  Part="1"
+AR Path="/5FBB8789" Ref="Q?"  Part="1"
+AR Path="/5FB8FF0F/5FBB8789" Ref="Q?"  Part="1"
+F 0 "Q?" V 7892 3350 50  0000 C CNN
+F 1 "SI3447CDV" V 7801 3350 50  0000 C CNN
+F 2 "BB:TSOP-6_1.5x3.0x0.95P" H 7750 3450 50  0001 C CNN
+F 3 "https://datasheet.lcsc.com/szlcsc/Vishay-Intertech-SI3447CDV-T1-E3_C145421.pdf" H 7550 3350 50  0001 C CNN
+F 4 "C145421" V 7550 3350 50  0001 C CNN "LCSC"
+	1    7550 3350
+	0    -1   -1   0
+$EndComp
+$Comp
+L Transistor_FET:2N7002 Q?
+U 1 1 5FBBD3A8
+P 7450 3750
+AR Path="/5F77B818/5FBBD3A8" Ref="Q?"  Part="1"
+AR Path="/5FA4C94D/5FBBD3A8" Ref="Q?"  Part="1"
+AR Path="/5FB8FF0F/5FBBD3A8" Ref="Q?"  Part="1"
+F 0 "Q?" H 7654 3796 50  0000 L CNN
+F 1 "2N7002" H 7654 3705 50  0000 L CNN
+F 2 "Package_TO_SOT_SMD:SOT-23" H 7650 3675 50  0001 L CIN
+F 3 "https://datasheet.lcsc.com/szlcsc/Changjiang-Electronics-Tech-CJ-CJ3134K_C110100.pdf" H 7450 3750 50  0001 L CNN
+F 4 "C8545" H 7450 3750 50  0001 C CNN "LCSC"
+	1    7450 3750
+	1    0    0    -1
+$EndComp
+$Comp
+L B.B-eagle-import:GND #GND?
+U 1 1 5FBC46B0
+P 7550 4050
+AR Path="/5FA4C94D/5FBC46B0" Ref="#GND?"  Part="1"
+AR Path="/5F9AAC80/5FBC46B0" Ref="#GND?"  Part="1"
+AR Path="/5FB8FF0F/5FBC46B0" Ref="#GND?"  Part="1"
+F 0 "#GND?" H 7550 4050 50  0001 C CNN
+F 1 "GND" H 7550 3970 59  0000 C CNN
+F 2 "" H 7550 4050 50  0001 C CNN
+F 3 "" H 7550 4050 50  0001 C CNN
+	1    7550 4050
+	1    0    0    -1
+$EndComp
+Wire Wire Line
+	7250 3750 7125 3750
+Wire Wire Line
+	7125 3750 7125 4150
+Wire Wire Line
+	7125 4150 4750 4150
+Wire Wire Line
+	4750 4150 4750 3625
+Connection ~ 4750 3625
+Wire Wire Line
+	7600 3550 7550 3550
+Connection ~ 7550 3550
+Wire Wire Line
+	7900 3550 7950 3550
+Wire Wire Line
+	7950 3550 7950 3250
+Wire Wire Line
+	7950 3250 7750 3250
+Wire Wire Line
+	8000 3250 7950 3250
+Connection ~ 7950 3250
+$Comp
+L Device:R R?
+U 1 1 5FBC9206
+P 7750 3550
+AR Path="/5F77B818/5FBC9206" Ref="R?"  Part="1"
+AR Path="/5FBC9206" Ref="R?"  Part="1"
+AR Path="/5FB8FF0F/5FBC9206" Ref="R?"  Part="1"
+F 0 "R?" V 7825 3425 50  0000 L CNN
+F 1 "1M" V 7825 3550 50  0000 L CNN
+F 2 "Resistor_SMD:R_0402_1005Metric" V 7680 3550 50  0001 C CNN
+F 3 "~" H 7750 3550 50  0001 C CNN
+F 4 "C26083" H 7750 3550 50  0001 C CNN "LCSC"
+	1    7750 3550
+	0    -1   -1   0
+$EndComp
 $EndSCHEMATC

Commit message: 18650
Parts:
- gave numbers to parts that had none: 11
Changed lines of the file:
@@
 $EndDescr
 $Comp
-L B.B-eagle-import:GND #GND?
+L B.B-eagle-import:GND #GND0104
 U 1 1 5FB90F26
 P 5975 3800
-F 0 "#GND?" H 5975 3800 50  0001 C CNN
+F 0 "#GND0104" H 5975 3800 50  0001 C CNN
 F 1 "GND" H 5975 3720 59  0000 C CNN
 F 2 "" H 5975 3800 50  0001 C CNN
@@
 BAT
 $Comp
-L Device:R R?
+L Device:R R48
 U 1 1 5FB9BA20
 P 6425 3750
-F 0 "R?" H 6355 3704 50  0000 R CNN
+F 0 "R48" H 6355 3704 50  0000 R CNN
 F 1 "1,2k" H 6355 3795 50  0000 R CNN
 F 2 "Resistor_SMD:R_0402_1005Metric" V 6355 3750 50  0001 C CNN
@@
 AR Path="/5FA4C94D/5FB9D127" Ref="#GND?"  Part="1"
 AR Path="/5F9AAC80/5FB9D127" Ref="#GND?"  Part="1"
-AR Path="/5FB8FF0F/5FB9D127" Ref="#GND?"  Part="1"
-F 0 "#GND?" H 6425 4000 50  0001 C CNN
+AR Path="/5FB8FF0F/5FB9D127" Ref="#GND0105"  Part="1"
+F 0 "#GND0105" H 6425 4000 50  0001 C CNN
 F 1 "GND" H 6425 3920 59  0000 C CNN
 F 2 "" H 6425 4000 50  0001 C CNN
@@
 AR Path="/5FA3274C/5FBFF4C4" Ref="LED?"  Part="1"
 AR Path="/5F9EE529/5FBFF4C4" Ref="LED?"  Part="1"
-AR Path="/5FB8FF0F/5FBFF4C4" Ref="LED?"  Part="1"
-F 0 "LED?" V 4900 3600 59  0000 L CNN
+AR Path="/5FB8FF0F/5FBFF4C4" Ref="LED4"  Part="1"
+F 0 "LED4" V 4900 3600 59  0000 L CNN
 F 1 "RED" V 5000 3275 59  0000 L CNN
 F 2 "LED_SMD:LED_0603_1608Metric" H 4900 3400 50  0001 C CNN
@@
 AR Path="/5FA3274C/5FC00D50" Ref="LED?"  Part="1"
 AR Path="/5F9EE529/5FC00D50" Ref="LED?"  Part="1"
-AR Path="/5FB8FF0F/5FC00D50" Ref="LED?"  Part="1"
-F 0 "LED?" V 4900 3825 59  0000 L CNN
+AR Path="/5FB8FF0F/5FC00D50" Ref="LED5"  Part="1"
+F 0 "LED5" V 4900 3825 59  0000 L CNN
 F 1 "BLUE" V 4725 3475 59  0000 L CNN
 F 2 "LED_SMD:LED_0603_1608Metric" H 4900 3625 50  0001 C CNN
@@
 	4750 3400 4750 3250
 $Comp
-L Device:R R?
+L Device:R R16
 U 1 1 5FC03C27
 P 5250 3400
-F 0 "R?" V 5300 3275 50  0000 R CNN
+F 0 "R16" V 5300 3275 50  0000 R CNN
 F 1 "1,2k" V 5325 3500 50  0000 R CNN
 F 2 "Resistor_SMD:R_0402_1005Metric" V 5180 3400 50  0001 C CNN
@@
 $EndComp
 $Comp
-L Device:R R?
+L Device:R R19
 U 1 1 5FC04CCC
 P 5250 3625
-F 0 "R?" V 5325 3850 50  0000 R CNN
+F 0 "R19" V 5325 3850 50  0000 R CNN
 F 1 "1,2k" V 5175 3700 50  0000 R CNN
 F 2 "Resistor_SMD:R_0402_1005Metric" V 5180 3625 50  0001 C CNN
@@
 AR Path="/5F9EE529/5FB1300F/5FB51226" Ref="C?"  Part="1"
 AR Path="/5FB26A97/5FB51226" Ref="C?"  Part="1"
-AR Path="/5FB8FF0F/5FB51226" Ref="C?"  Part="1"
-F 0 "C?" H 6990 3496 50  0000 L CNN
+AR Path="/5FB8FF0F/5FB51226" Ref="C76"  Part="1"
+F 0 "C76" H 6990 3496 50  0000 L CNN
 F 1 "1uf" H 6990 3405 50  0000 L CNN
 F 2 "Resistor_SMD:R_0402_1005Metric" H 6913 3300 50  0001 C CNN
@@
 AR Path="/5F9EE529/5FB1300F/5FB5121E" Ref="#GND?"  Part="1"
 AR Path="/5FB26A97/5FB5121E" Ref="#GND?"  Part="1"
-AR Path="/5FB8FF0F/5FB5121E" Ref="#GND?"  Part="1"
-F 0 "#GND?" H 6875 3700 50  0001 C CNN
+AR Path="/5FB8FF0F/5FB5121E" Ref="#GND0107"  Part="1"
+F 0 "#GND0107" H 6875 3700 50  0001 C CNN
 F 1 "GND" H 6875 3620 59  0000 C CNN
 F 2 "" H 6875 3700 50  0001 C CNN
@@
 	6875 3250 7350 3250
 $Comp
-L B.B-rescue:SE9017 U?
+L B.B-rescue:SE9017 U72
 U 1 1 5FB4881E
 P 5975 3250
-F 0 "U?" H 5950 3475 50  0000 C CNN
+F 0 "U72" H 5950 3475 50  0000 C CNN
 F 1 "SE9017" H 5950 3384 50  0000 C CNN
 F 2 "Package_SO:SOP-8_3.76x4.96mm_P1.27mm" H 5975 3250 50  0001 C CNN
@@
 AR Path="/5F9EE529/5FB1300F/5FB55492" Ref="C?"  Part="1"
 AR Path="/5FB26A97/5FB55492" Ref="C?"  Part="1"
-AR Path="/5FB8FF0F/5FB55492" Ref="C?"  Part="1"
-F 0 "C?" H 4290 3521 50  0000 L CNN
+AR Path="/5FB8FF0F/5FB55492" Ref="C77"  Part="1"
+F 0 "C77" H 4290 3521 50  0000 L CNN
 F 1 "1uf" H 4290 3430 50  0000 L CNN
 F 2 "Resistor_SMD:R_0402_1005Metric" H 4213 3325 50  0001 C CNN
@@
 AR Path="/5F9EE529/5FB1300F/5FB55498" Ref="#GND?"  Part="1"
 AR Path="/5FB26A97/5FB55498" Ref="#GND?"  Part="1"
-AR Path="/5FB8FF0F/5FB55498" Ref="#GND?"  Part="1"
-F 0 "#GND?" H 4175 3725 50  0001 C CNN
+AR Path="/5FB8FF0F/5FB55498" Ref="#GND0155"  Part="1"
+F 0 "#GND0155" H 4175 3725 50  0001 C CNN
 F 1 "GND" H 4175 3645 59  0000 C CNN
 F 2 "" H 4175 3725 50  0001 C CNN
@@
 AR Path="/5FA4C94D/5FBB8789" Ref="Q?"  Part="1"
 AR Path="/5FBB8789" Ref="Q?"  Part="1"
-AR Path="/5FB8FF0F/5FBB8789" Ref="Q?"  Part="1"
-F 0 "Q?" V 7892 3350 50  0000 C CNN
+AR Path="/5FB8FF0F/5FBB8789" Ref="Q11"  Part="1"
+F 0 "Q11" V 7892 3350 50  0000 C CNN
 F 1 "SI3447CDV" V 7801 3350 50  0000 C CNN
 F 2 "BB:TSOP-6_1.5x3.0x0.95P" H 7750 3450 50  0001 C CNN
@@
 AR Path="/5F77B818/5FBBD3A8" Ref="Q?"  Part="1"
 AR Path="/5FA4C94D/5FBBD3A8" Ref="Q?"  Part="1"
-AR Path="/5FB8FF0F/5FBBD3A8" Ref="Q?"  Part="1"
-F 0 "Q?" H 7654 3796 50  0000 L CNN
+AR Path="/5FB8FF0F/5FBBD3A8" Ref="Q12"  Part="1"
+F 0 "Q12" H 7654 3796 50  0000 L CNN
 F 1 "2N7002" H 7654 3705 50  0000 L CNN
 F 2 "Package_TO_SOT_SMD:SOT-23" H 7650 3675 50  0001 L CIN
@@
 AR Path="/5FA4C94D/5FBC46B0" Ref="#GND?"  Part="1"
 AR Path="/5F9AAC80/5FBC46B0" Ref="#GND?"  Part="1"
-AR Path="/5FB8FF0F/5FBC46B0" Ref="#GND?"  Part="1"
-F 0 "#GND?" H 7550 4050 50  0001 C CNN
+AR Path="/5FB8FF0F/5FBC46B0" Ref="#GND0156"  Part="1"
+F 0 "#GND0156" H 7550 4050 50  0001 C CNN
 F 1 "GND" H 7550 3970 59  0000 C CNN
 F 2 "" H 7550 4050 50  0001 C CNN
@@
 AR Path="/5F77B818/5FBC9206" Ref="R?"  Part="1"
 AR Path="/5FBC9206" Ref="R?"  Part="1"
-AR Path="/5FB8FF0F/5FBC9206" Ref="R?"  Part="1"
-F 0 "R?" V 7825 3425 50  0000 L CNN
+AR Path="/5FB8FF0F/5FBC9206" Ref="R17"  Part="1"
+F 0 "R17" V 7825 3425 50  0000 L CNN
 F 1 "1M" V 7825 3550 50  0000 L CNN
 F 2 "Resistor_SMD:R_0402_1005Metric" V 7680 3550 50  0001 C CNN

Commit message: polifuse
-filtr k prijmaci IR
-merwni bterky -> za zapinani
-odstraneni odpojovani nabijecky + oprava napajeciho prouhu
-odstraneni prevodniku napeti k WS2812
Parts:
- removed Q11: SI3447CDV, BB:TSOP-6_1.5x3.0x0.95P, symbol B.B-rescue:Q_PMOS_DSG
- removed Q12: 2N7002, Package_TO_SOT_SMD:SOT-23, symbol Transistor_FET:2N7002
- removed R17: 1M, Resistor_SMD:R_0402_1005Metric, symbol Device:R
- R16, R19: value 1,2k -> 1k; LCSC C25862 -> C11702
- R48: value 1,2k -> 2k; LCSC C25862 -> https://datasheet.lcsc.com/szlcsc/Seaward-Elec-SE9017-HF_C1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
- U72: footprint Package_SO:SOP-8_3.76x4.96mm_P1.27mm -> Package_TO_SOT_SMD:SOT-23-6; LCSC C115752 -> C115751
Connections:
- wire segments 26 -> 17
Changed lines of the file:
@@
 $Descr A4 11693 8268
 encoding utf-8
-Sheet 7 8
+Sheet 5 8
 Title ""
 Date ""
@@
 Wire Wire Line
 	4100 3250 4175 3250
-Text HLabel 8000 3250 2    50   Input ~ 0
+Text HLabel 6975 3250 2    50   Input ~ 0
 BAT
 $Comp
@@
 P 6425 3750
 F 0 "R48" H 6355 3704 50  0000 R CNN
-F 1 "1,2k" H 6355 3795 50  0000 R CNN
+F 1 "2k" H 6355 3795 50  0000 R CNN
 F 2 "Resistor_SMD:R_0402_1005Metric" V 6355 3750 50  0001 C CNN
 F 3 "~" H 6425 3750 50  0001 C CNN
-F 4 "C25862" V 6425 3750 50  0001 C CNN "LCSC"
+F 4 "https://datasheet.lcsc.com/szlcsc/Seaward-Elec-SE9017-HF_C115752.pdf" V 6425 3750 50  0001 C CNN "LCSC"
 	1    6425 3750
 	-1   0    0    1
@@
 Wire Wire Line
 	4750 3400 4750 3250
-$Comp
-L Device:R R16
-U 1 1 5FC03C27
-P 5250 3400
-F 0 "R16" V 5300 3275 50  0000 R CNN
-F 1 "1,2k" V 5325 3500 50  0000 R CNN
-F 2 "Resistor_SMD:R_0402_1005Metric" V 5180 3400 50  0001 C CNN
-F 3 "~" H 5250 3400 50  0001 C CNN
-F 4 "C25862" V 5250 3400 50  0001 C CNN "LCSC"
-	1    5250 3400
-	0    -1   -1   0
-$EndComp
-$Comp
-L Device:R R19
-U 1 1 5FC04CCC
-P 5250 3625
-F 0 "R19" V 5325 3850 50  0000 R CNN
-F 1 "1,2k" V 5175 3700 50  0000 R CNN
-F 2 "Resistor_SMD:R_0402_1005Metric" V 5180 3625 50  0001 C CNN
-F 3 "~" H 5250 3625 50  0001 C CNN
-F 4 "C25862" V 5250 3625 50  0001 C CNN "LCSC"
-	1    5250 3625
-	0    1    1    0
-$EndComp
 $Comp
 L Device:C C?
@@
 Connection ~ 6875 3250
 Wire Wire Line
-	6875 3250 7350 3250
+	6875 3250 6975 3250
 $Comp
 L B.B-rescue:SE9017 U72
@@
 F 0 "U72" H 5950 3475 50  0000 C CNN
 F 1 "SE9017" H 5950 3384 50  0000 C CNN
-F 2 "Package_SO:SOP-8_3.76x4.96mm_P1.27mm" H 5975 3250 50  0001 C CNN
+F 2 "Package_TO_SOT_SMD:SOT-23-6" H 5975 3250 50  0001 C CNN
 F 3 "https://datasheet.lcsc.com/szlcsc/Seaward-Elec-SE9017-HF_C115752.pdf" H 5975 3250 50  0001 C CNN
-F 4 "C115752" H 5975 3250 50  0001 C CNN "LCSC"
+F 4 "C115751" H 5975 3250 50  0001 C CNN "LCSC"
 	1    5975 3250
 	1    0    0    -1
@@
 	4175 3250 4750 3250
 $Comp
-L B.B-rescue:Q_PMOS_DSG Q?
-U 1 1 5FBB8789
-P 7550 3350
-AR Path="/5F9EE529/5FBB8789" Ref="Q?"  Part="1"
-AR Path="/5FA4C94D/5FBB8789" Ref="Q?"  Part="1"
-AR Path="/5FBB8789" Ref="Q?"  Part="1"
-AR Path="/5FB8FF0F/5FBB8789" Ref="Q11"  Part="1"
-F 0 "Q11" V 7892 3350 50  0000 C CNN
-F 1 "SI3447CDV" V 7801 3350 50  0000 C CNN
-F 2 "BB:TSOP-6_1.5x3.0x0.95P" H 7750 3450 50  0001 C CNN
-F 3 "https://datasheet.lcsc.com/szlcsc/Vishay-Intertech-SI3447CDV-T1-E3_C145421.pdf" H 7550 3350 50  0001 C CNN
-F 4 "C145421" V 7550 3350 50  0001 C CNN "LCSC"
-	1    7550 3350
+L Device:R R16
+U 1 1 5FC03C27
+P 5250 3400
+F 0 "R16" V 5300 3275 50  0000 R CNN
+F 1 "1k" V 5325 3500 50  0000 R CNN
+F 2 "Resistor_SMD:R_0402_1005Metric" V 5180 3400 50  0001 C CNN
+F 3 "~" H 5250 3400 50  0001 C CNN
+F 4 "C11702" V 5250 3400 50  0001 C CNN "LCSC"
+	1    5250 3400
 	0    -1   -1   0
 $EndComp
 $Comp
-L Transistor_FET:2N7002 Q?
-U 1 1 5FBBD3A8
-P 7450 3750
-AR Path="/5F77B818/5FBBD3A8" Ref="Q?"  Part="1"
-AR Path="/5FA4C94D/5FBBD3A8" Ref="Q?"  Part="1"
-AR Path="/5FB8FF0F/5FBBD3A8" Ref="Q12"  Part="1"
-F 0 "Q12" H 7654 3796 50  0000 L CNN
-F 1 "2N7002" H 7654 3705 50  0000 L CNN
-F 2 "Package_TO_SOT_SMD:SOT-23" H 7650 3675 50  0001 L CIN
-F 3 "https://datasheet.lcsc.com/szlcsc/Changjiang-Electronics-Tech-CJ-CJ3134K_C110100.pdf" H 7450 3750 50  0001 L CNN
-F 4 "C8545" H 7450 3750 50  0001 C CNN "LCSC"
-	1    7450 3750
-	1    0    0    -1
-$EndComp
-$Comp
-L B.B-eagle-import:GND #GND?
-U 1 1 5FBC46B0
-P 7550 4050
-AR Path="/5FA4C94D/5FBC46B0" Ref="#GND?"  Part="1"
-AR Path="/5F9AAC80/5FBC46B0" Ref="#GND?"  Part="1"
-AR Path="/5FB8FF0F/5FBC46B0" Ref="#GND0156"  Part="1"
-F 0 "#GND0156" H 7550 4050 50  0001 C CNN
-F 1 "GND" H 7550 3970 59  0000 C CNN
-F 2 "" H 7550 4050 50  0001 C CNN
-F 3 "" H 7550 4050 50  0001 C CNN
-	1    7550 4050
-	1    0    0    -1
-$EndComp
-Wire Wire Line
-	7250 3750 7125 3750
-Wire Wire Line
-	7125 3750 7125 4150
-Wire Wire Line
-	7125 4150 4750 4150
-Wire Wire Line
-	4750 4150 4750 3625
-Connection ~ 4750 3625
-Wire Wire Line
-	7600 3550 7550 3550
-Connection ~ 7550 3550
-Wire Wire Line
-	7900 3550 7950 3550
-Wire Wire Line
-	7950 3550 7950 3250
-Wire Wire Line
-	7950 3250 7750 3250
-Wire Wire Line
-	8000 3250 7950 3250
-Connection ~ 7950 3250
-$Comp
-L Device:R R?
-U 1 1 5FBC9206
-P 7750 3550
-AR Path="/5F77B818/5FBC9206" Ref="R?"  Part="1"
-AR Path="/5FBC9206" Ref="R?"  Part="1"
-AR Path="/5FB8FF0F/5FBC9206" Ref="R17"  Part="1"
-F 0 "R17" V 7825 3425 50  0000 L CNN
-F 1 "1M" V 7825 3550 50  0000 L CNN
-F 2 "Resistor_SMD:R_0402_1005Metric" V 7680 3550 50  0001 C CNN
-F 3 "~" H 7750 3550 50  0001 C CNN
-F 4 "C26083" H 7750 3550 50  0001 C CNN "LCSC"
-	1    7750 3550
-	0    -1   -1   0
+L Device:R R19
+U 1 1 5FC04CCC
+P 5250 3625
+F 0 "R19" V 5325 3850 50  0000 R CNN
+F 1 "1k" V 5175 3600 50  0000 R CNN
+F 2 "Resistor_SMD:R_0402_1005Metric" V 5180 3625 50  0001 C CNN
+F 3 "~" H 5250 3625 50  0001 C CNN
+F 4 "C11702" V 5250 3625 50  0001 C CNN "LCSC"
+	1    5250 3625
+	0    1    1    0
 $EndComp
 $EndSCHEMATC

Commit message: napajeni_na_stejne_strane
-poradi na konektoru
-napajeni IR prijmece z 5V na VCC
-vyssi nabijeci proud
-WS2812_power na IO21
Parts:
- R48: value 2k -> 1.5k; footprint Resistor_SMD:R_0402_1005Metric -> Resistor_SMD:R_0603_1608Metric; LCSC https://datasheet.lcsc.com/szlcsc/Seaward-Elec-SE9017-HF_C1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 -> C22843
Changed lines of the file:
@@
 $Descr A4 11693 8268
 encoding utf-8
-Sheet 5 8
+Sheet 3 8
 Title ""
 Date ""
@@
 P 6425 3750
 F 0 "R48" H 6355 3704 50  0000 R CNN
-F 1 "2k" H 6355 3795 50  0000 R CNN
-F 2 "Resistor_SMD:R_0402_1005Metric" V 6355 3750 50  0001 C CNN
+F 1 "1.5k" H 6355 3795 50  0000 R CNN
+F 2 "Resistor_SMD:R_0603_1608Metric" V 6355 3750 50  0001 C CNN
 F 3 "~" H 6425 3750 50  0001 C CNN
-F 4 "https://datasheet.lcsc.com/szlcsc/Seaward-Elec-SE9017-HF_C115752.pdf" V 6425 3750 50  0001 C CNN "LCSC"
+F 4 "C22843" V 6425 3750 50  0001 C CNN "LCSC"
 	1    6425 3750
 	-1   0    0    1

Commit message: popisky
-popisky
-poladeni uddeleni enkoderu
-poladeni nayvu drah
-priopjeni gnd USB
-poligon V5 na led-desce do spodni vrstvu
Parts:
- C76, C77: symbol Device:C -> B.B-rescue:C-Device
- R16, R19, R48: symbol Device:R -> B.B-rescue:R-Device

Commit message: LDC footprint
prodlouzeni pedu pro usnadneni rucniho osazovani
Parts:
- C76, C77: symbol B.B-rescue:C-Device -> B.B-rescue:C-Device-B.B-rescue
- LED4, LED5: symbol B.B-eagle-import:LED -> B.B-rescue:LED-B.B-eagle-import
- R16, R19, R48: symbol B.B-rescue:R-Device -> B.B-rescue:R-Device-B.B-rescue
- U72: symbol B.B-rescue:SE9017 -> B.B-rescue:SE9017-B.B-rescue
Changed lines of the file:
@@
 	3900 3400 3975 3400
 $Comp
-L B.B-eagle-import:LED LED?
+L B.B-rescue:LED-B.B-eagle-import LED?
 U 1 1 5FBFF4C4
 P 4700 3550
@@
 $EndComp
 $Comp
-L B.B-eagle-import:LED LED?
+L B.B-rescue:LED-B.B-eagle-import LED?
 U 1 1 5FC00D50
 P 4700 3775
@@
 	4550 3550 4550 3400
 $Comp
-L B.B-rescue:C-Device C?
+L B.B-rescue:C-Device-B.B-rescue C?
 U 1 1 5FB55492
 P 3975 3625
@@
 $EndComp
 $Comp
-L B.B-eagle-import:GND #GND?
+L B.B-rescue:GND-B.B-eagle-import #GND?
 U 1 1 5FB55498
 P 3975 3875
@@
 	3975 3400 4550 3400
 $Comp
-L B.B-rescue:R-Device R16
+L B.B-rescue:R-Device-B.B-rescue R16
 U 1 1 5FC03C27
 P 5050 3550
@@
 $EndComp
 $Comp
-L B.B-rescue:R-Device R19
+L B.B-rescue:R-Device-B.B-rescue R19
 U 1 1 5FC04CCC
 P 5050 3775
@@
 $EndComp
 $Comp
-L B.B-eagle-import:GND #GND0104
+L B.B-rescue:GND-B.B-eagle-import #GND0104
 U 1 1 5FB90F26
 P 5775 3950
@@
 $EndComp
 $Comp
-L B.B-eagle-import:GND #GND?
+L B.B-rescue:GND-B.B-eagle-import #GND?
 U 1 1 5FB9D127
 P 6225 4150
@@
 $EndComp
 $Comp
-L B.B-rescue:R-Device R48
+L B.B-rescue:R-Device-B.B-rescue R48
 U 1 1 5FB9BA20
 P 6225 3900
@@
 	5200 3550 5325 3550
 $Comp
-L B.B-rescue:SE9017 U72
+L B.B-rescue:SE9017-B.B-rescue U72
 U 1 1 5FB4881E
 P 5775 3400
@@
 	6675 3450 6675 3400
 $Comp
-L B.B-eagle-import:GND #GND?
+L B.B-rescue:GND-B.B-eagle-import #GND?
 U 1 1 5FB5121E
 P 6675 3850
@@
 $EndComp
 $Comp
-L B.B-rescue:C-Device C?
+L B.B-rescue:C-Device-B.B-rescue C?
 U 1 1 5FB51226
 P 6675 3600

Commit message: JLCdata
- korekce pozice a natoceni
- data pro vyrobu
Parts:
- U72: JLCPCB_CORRECTION (none) -> 0;0;180
Changed lines of the file:
@@
 $Descr A4 11693 8268
 encoding utf-8
-Sheet 8 8
+Sheet 7 8
 Title ""
 Date ""
@@
 F 3 "https://datasheet.lcsc.com/szlcsc/Seaward-Elec-SE9017-HF_C115752.pdf" H 5775 3400 50  0001 C CNN
 F 4 "C115751" H 5775 3400 50  0001 C CNN "LCSC"
+F 5 "0;0;180" H 5775 3400 50  0001 C CNN "JLCPCB_CORRECTION"
 	1    5775 3400
 	1    0    0    -1
