File: main_board/B.B/HlavniDeska.kicad_pcb (KiCad board)
At the start: 4 copper layers, 98 x 98 mm, 122 parts, among them J1 Conn_01x04, J2 Conn_01x11, J4 Conn_01x04, J5 USB_C_Receptacle_USB2.0, J6 Conn_01x04-Connector_Generic-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, M1 Motor_DC, Q1 2N7002, Q10 2N7002, Q11 SI3447CDV, Q2 2N7002, Q3 AO3400A, Q5 SI3447CDV, Q7 SI3447CDV, SW1 SW_DIP_x01, SW2 SW_DIP_x01, SW3 SW_DIP_x01, SW4 SW_DIP_x02, SW5 SW_DIP_x01, U61 BMX055, U62 LD39200, U63 FP6276, U64 CP2102N-A01-GQFN28, U65 ESP32-WROVER, U67 M41T62, U68 IRM-H936, U69 SPL06, U70 MH253ESO, U71 MH253ESO, U72 SE9017, U73 MPU6050, U74 QMC5883, Y1 32.768kHz

Commit message: presuny_konektoru
Parts:
- removed C114, C94: 2.2uf, Capacitor_SMD:C_0805_2012Metric
- removed C71, C73: 22n, Capacitor_SMD:C_0402_1005Metric
- removed C72, C74: 18p/50V, Capacitor_SMD:C_0402_1005Metric
- removed C81: 0.1uf, Resistor_SMD:R_0402_1005Metric
- removed C85: 1uf, Resistor_SMD:R_0402_1005Metric
- removed C86: 220nf, Capacitor_SMD:C_0402_1005Metric
- removed D2: D, BB:SOD-323
- removed J4: Conn_01x04, Connector_PinSocket_2.54mm:PinSocket_1x04_P2.54mm_Vertical
- removed J6: Conn_01x04-Connector_Generic-B.B-rescue, Connector_PinHeader_2.54mm:PinHeader_1x04_P2.54mm_Vertical
- removed LED3: IR, LED_SMD:LED_0603_1608Metric
- removed R43: 220, Resistor_SMD:R_0402_1005Metric
- removed R45: 100k, Resistor_SMD:R_0402_1005Metric
- removed R46, R47: 47k, Resistor_SMD:R_0402_1005Metric
- removed U68: IRM-H936, BB:SMD-4_4.0x5.0x2.54P
- removed U70: MH253ESO, Package_TO_SOT_SMD:SOT-23
- removed U74: QMC5883, Package_LGA:LGA-16_3x3mm_P0.5mm
- added D1: SS54, BB:DO-214AC, F.Cu at (211.0, 91.8)
- added J10: Conn_01x03, Connector_PinHeader_2.54mm:PinHeader_1x03_P2.54mm_Vertical, F.Cu at (204.4, 65.3)
- added J11: Conn_01x03, Connector_PinHeader_2.54mm:PinHeader_1x03_P2.54mm_Vertical, F.Cu at (184.6, 60.3)
- added J12: Conn_01x03, Connector_PinHeader_2.54mm:PinHeader_1x03_P2.54mm_Vertical, F.Cu at (208.0, 65.3)
- added J13: Conn_01x03, Connector_PinHeader_2.54mm:PinHeader_1x03_P2.54mm_Vertical, F.Cu at (188.2, 60.3)
- added J14: Conn_01x03, Connector_PinHeader_2.54mm:PinHeader_1x03_P2.54mm_Vertical, F.Cu at (211.6, 65.3)
- added J15: Conn_01x03, Connector_PinHeader_2.54mm:PinHeader_1x03_P2.54mm_Vertical, F.Cu at (191.8, 60.3)
- added J8: Conn_01x03, Connector_PinHeader_2.54mm:PinHeader_1x03_P2.54mm_Vertical, F.Cu at (200.8, 65.3)
- added J9: Conn_01x03, Connector_PinHeader_2.54mm:PinHeader_1x03_P2.54mm_Vertical, F.Cu at (195.4, 60.3)
- added Q4: 2N7002, Package_TO_SOT_SMD:SOT-23, F.Cu at (211.0, 98.2)
- added R11: 220, Resistor_SMD:R_0402_1005Metric, F.Cu at (215.4, 103.8)
- added R12: 12k, Resistor_SMD:R_0402_1005Metric, F.Cu at (197.7, 62.9)
- added R17: 12k, Resistor_SMD:R_0402_1005Metric, F.Cu at (182.0, 62.8)
- added R39: 12k, Resistor_SMD:R_0402_1005Metric, F.Cu at (186.4, 67.7)
- added R40: 12k, Resistor_SMD:R_0402_1005Metric, F.Cu at (193.6, 67.7)
- added R9: 47k, Resistor_SMD:R_0402_1005Metric, F.Cu at (211.0, 101.3)
- C67: value 10uf -> 2.2uf; footprint Resistor_SMD:R_0805_2012Metric -> Capacitor_SMD:C_0402_1005Metric
- C68: value 0.1uf -> 2.2uf; footprint Capacitor_SMD:C_0805_2012Metric -> Capacitor_SMD:C_0402_1005Metric
- J1: footprint Connector_PinSocket_2.54mm:PinSocket_1x04_P2.54mm_Vertical -> Connector_PinHeader_2.54mm:PinHeader_1x04_P2.54mm_Vertical
- JP1, JP2: footprint Jumper:SolderJumper-3_P1.3mm_Open_RoundedPad1.0x1.5mm -> Jumper:SolderJumper-3_P1.3mm_Bridged12_RoundedPad1.0x1.5mm_NumberLabels
- R5: value 470 -> 12k
- U61: value BMX055 -> QMC6310; footprint BB:LGA_4.5x3 -> BB:QMC6310
- U71: value MH253ESO -> piezo; footprint Package_TO_SOT_SMD:SOT-23 -> BB:piezo
- moved J1 73.2 mm to (216.4, 122.2)
- moved C104 54.6 mm to (231.5, 133.1)
- moved SW1 54.0 mm to (225.8, 133.0)
- moved R20 41.8 mm to (220.3, 137.0), turned to 90 degrees
- moved R5 33.7 mm to (175.5, 124.0), turned to 180 degrees
- moved U71 24.3 mm to (176.1, 73.0), turned to 90 degrees
- moved C68 15.2 mm to (182.7, 123.8), turned to 270 degrees
- moved U61 8.78 mm to (174.2, 136.5), turned to 0 degrees
- moved C67 6.27 mm to (172.0, 136.6), turned to 270 degrees
- moved SW3 2.40 mm to (225.9, 111.2)
- moved SW5 2.31 mm to (225.8, 118.4)
- moved C107 2.21 mm to (220.3, 125.7)
- moved Q10 1.86 mm to (217.9, 68.7)
- moved Q7 1.86 mm to (218.9, 72.3)
- moved R41 1.86 mm to (216.8, 72.3)
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Connections:
- C62 pad 1: /ESP3200/IO5-up -> Net-(C62-Pad1)
- C68 pad 1: +3V3 -> Net-(C68-Pad1)
- J1 pad 1: GND -> VCC
- J1 pad 2: +3V3 -> /expanz00/A9-TX
- J1 pad 3: /expanz00/ENC_OUT_0 -> /expanz00/A9-RX
- J1 pad 4: /expanz00/ENC_OUT_1 -> GND
- J2 pad 5: /ESP3200/IO0-up -> Net-(J2-Pad5)
- J5 pad B12: (no net) -> GND
- J5 pad S1: (no net) -> Net-(J5-PadS1)
- Q1 pad 1: /ESP3200/IO5-up -> Net-(C62-Pad1)
- R5 pad 1: Net-(C114-Pad1) -> /ESP3200/IO34
- R5 pad 2: Net-(D2-Pad1) -> +3V3
- R8 pad 1: /ESP3200/IO5-up -> Net-(C62-Pad1)
- SW5 pad 2: /ESP3200/IO5-up -> Net-(C62-Pad1)
- U65 pad 16: /expanz00/ENC_OUT_1 -> /ESP3200/IO13
- U65 pad 26: /expanz00/ENC_OUT_0 -> /ESP3200/IO4
- U65 pad 8: /ESP3200/IO32 -> /expanz00/A9-RX
- U65 pad 9: /ESP3200/IO33 -> /expanz00/A9-TX
- U69 pad 5: /ESP3200/IO27 -> /perception00/int_baro
- U71 pad 1: +3V3 -> Net-(D1-Pad2)
- U71 pad 2: /expanz00/ENC_OUT_1 -> VCC
- U73 pad 20: Net-(C94-Pad1) -> Net-(C68-Pad1)
Routing:
- net /expanz00/ENC_OUT_1: track 103.7 -> 0.00 mm, vias 4 -> 0
- net /expanz00/ENC_OUT_0: track 87.2 -> 0.00 mm, vias 1 -> 0
- net VCC: track 76.9 -> 153.0 mm, vias 3 -> 5
- net /ESP3200/IO4: track 0.00 -> 74.3 mm, vias 0 -> 1
- net /ESP3200/IO32: track 64.1 -> 0.00 mm, vias 3 -> 0
- net /ESP3200/IO33: track 63.7 -> 0.00 mm, vias 3 -> 0
- net /ESP3200/IO13: track 0.00 -> 63.7 mm, vias 0 -> 1
- net /ESP3200/IO15-up: track 24.1 -> 82.8 mm
- net Net-(D1-Pad2): track 0.00 -> 50.3 mm, vias 0 -> 2
- net /ESP3200/IO35: track 30.5 -> 76.5 mm
- net /ESP3200/IO21: track 0.00 -> 44.7 mm
- net +3V3: track 74.7 -> 31.1 mm, vias 21 -> 24
- net /ESP3200/IO2-down: track 30.9 -> 73.6 mm, vias 0 -> 1
- net /ESP3200/IO0-up: track 76.7 -> 114.4 mm, vias 3 -> 5
- net GND: track 122.1 -> 85.5 mm, vias 46 -> 40
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Other:
- outline, holes or cut-outs redrawn
- board text removed: "ENC0"
- board text removed: "ENC1"
