File: main_board/B.B/expanz.sch (KiCad schematic (older format))
At the start: 25 parts, among them J1 Conn_01x04, J4 Conn_01x04, M1 Motor_DC, Q10 2N7002, Q7 SI3447CDV, Q8 2N7002, Q9 SI3447CDV, U68 IRM-H936, U70 MH253ESO, U71 MH253ESO

Commit message: lucerna
Parts:
- removed C73: 22n, Capacitor_SMD:C_0402_1005Metric, symbol B.B-rescue:C-Device-B.B-rescue
- removed C74: 18p/50V, Capacitor_SMD:C_0402_1005Metric, symbol B.B-rescue:C-Device-B.B-rescue
- removed Q8: 2N7002, Package_TO_SOT_SMD:SOT-23, symbol B.B-rescue:2N7002-Transistor_FET-B.B-rescue
- removed Q9: SI3447CDV, BB:TSOP-6_1.5x3.0x0.95P, symbol B.B-rescue:Q_PMOS_DSG-B.B-rescue
- removed R42: 100k, Resistor_SMD:R_0402_1005Metric, symbol B.B-rescue:R-Device-B.B-rescue
- removed R47: 47k, Resistor_SMD:R_0402_1005Metric, symbol B.B-rescue:R-Device-B.B-rescue
- removed U71: MH253ESO, Package_TO_SOT_SMD:SOT-23, symbol B.B-rescue:MH253ESO-B.B-rescue
- added D1: SS54, BB:DO-214AC, symbol B.B-rescue:D_Schottky-Device-B.B-rescue
- added Q4: 2N7002, Package_TO_SOT_SMD:SOT-23, symbol B.B-rescue:2N7002-Transistor_FET-B.B-rescue
- added R9: 47k, Resistor_SMD:R_0402_1005Metric, symbol B.B-rescue:R-Device-B.B-rescue
- added U71: piezo, BB:piezo, symbol B.B-rescue:piezo
- M1: footprint Connector_PinHeader_1.00mm:PinHeader_1x02_P1.00mm_Vertical -> Connector_JST:JST_EH_B2B-EH-A_1x02_P2.50mm_Vertical
Connections:
- net VCC: now also D1.1 (K), U71.2 (+)
- net ENC_OUT_1: no longer names the net of J4.4 (Pin_4)
- net ENC_OUT_1: no longer J1.4 (Pin_4)
- new net: D1.2 (A), Q4.3 (D), U71.1 (-)
- new net piezo: Q4.1 (G), R9.1
Other:
- moved on the sheet: C71, C72, J1, J4, R46, U70

Commit message: presuny_konektoru
Parts:
- removed C114: 2.2uf, Capacitor_SMD:C_0805_2012Metric, symbol B.B-rescue:C-Device-B.B-rescue
- removed C71: 22n, Capacitor_SMD:C_0402_1005Metric, symbol B.B-rescue:C-Device-B.B-rescue
- removed C72: 18p/50V, Capacitor_SMD:C_0402_1005Metric, symbol B.B-rescue:C-Device-B.B-rescue
- removed C81: 0.1uf, Resistor_SMD:R_0402_1005Metric, symbol B.B-rescue:C-Device-B.B-rescue
- removed D2: D, BB:SOD-323, symbol B.B-rescue:D-Device-B.B-rescue
- removed J1, J4: Conn_01x04, Connector_PinSocket_2.54mm:PinSocket_1x04_P2.54mm_Vertical, symbol B.B-rescue:Conn_01x04-Connector_Generic-B.B-rescue
- removed LED3: IR, LED_SMD:LED_0603_1608Metric, symbol B.B-rescue:LED-B.B-eagle-import
- removed R43: 220, Resistor_SMD:R_0402_1005Metric, symbol B.B-rescue:R-Device-B.B-rescue
- removed R46: 47k, Resistor_SMD:R_0402_1005Metric, symbol B.B-rescue:R-Device-B.B-rescue
- removed R5: 470, Resistor_SMD:R_0402_1005Metric, symbol B.B-rescue:R-Device-B.B-rescue
- removed U68: IRM-H936, BB:SMD-4_4.0x5.0x2.54P, symbol B.B-rescue:IRM-H936-B.B-rescue
- removed U70: MH253ESO, Package_TO_SOT_SMD:SOT-23, symbol B.B-rescue:MH253ESO-B.B-rescue
- added J1: Conn_01x04, Connector_PinHeader_2.54mm:PinHeader_1x04_P2.54mm_Vertical, symbol Connector_Generic:Conn_01x04
Connections:
- net VCC: now also J1.1 (Pin_1)
- new net A9-RX: J1.3 (Pin_3)
- new net A9-TX: J1.2 (Pin_2)
Other:
- note added: "conn for A9G"
- moved on the sheet: D1, D3, M1, Q10, Q4, Q7, R41, R9, U71
