File: main_board/B.B/servos.sch (KiCad schematic (older format))
At the start: 8 parts, among them J10 Conn_01x03, J11 Conn_01x03, J12 Conn_01x03, J13 Conn_01x03, J14 Conn_01x03, J15 Conn_01x03, J8 Conn_01x03, J9 Conn_01x03

Commit message: posouvani-LCSC
Parts:
- J10, J11, J12, J13, J14, J15, J8, J9: LCSC (none) -> C376076
Connections:
- net T0: now also J9.3 (Pin_3); no longer J9.2 (Pin_2)
- net T1: now also J11.3 (Pin_3); no longer J11.2 (Pin_2)
- net T2: now also J13.3 (Pin_3); no longer J13.2 (Pin_2)
- net T3: now also J15.3 (Pin_3); no longer J15.2 (Pin_2)
- new net: J11.2 (Pin_2), J13.2 (Pin_2), J15.2 (Pin_2), J9.2 (Pin_2)
Changed lines of the file:
@@
 F 2 "Connector_PinHeader_2.54mm:PinHeader_1x03_P2.54mm_Vertical" H 5075 3225 50  0001 C CNN
 F 3 "~" H 5075 3225 50  0001 C CNN
+F 4 "C376076 " H 5075 3225 50  0001 C CNN "LCSC"
 	1    5075 3225
 	1    0    0    -1
@@
 F 2 "Connector_PinHeader_2.54mm:PinHeader_1x03_P2.54mm_Vertical" H 5075 3550 50  0001 C CNN
 F 3 "~" H 5075 3550 50  0001 C CNN
+F 4 "C376076 " H 5075 3550 50  0001 C CNN "LCSC"
 	1    5075 3550
 	1    0    0    -1
@@
 F 2 "Connector_PinHeader_2.54mm:PinHeader_1x03_P2.54mm_Vertical" H 5075 3875 50  0001 C CNN
 F 3 "~" H 5075 3875 50  0001 C CNN
+F 4 "C376076 " H 5075 3875 50  0001 C CNN "LCSC"
 	1    5075 3875
 	1    0    0    -1
@@
 F 2 "Connector_PinHeader_2.54mm:PinHeader_1x03_P2.54mm_Vertical" H 5075 4200 50  0001 C CNN
 F 3 "~" H 5075 4200 50  0001 C CNN
+F 4 "C376076" H 5075 4200 50  0001 C CNN "LCSC"
 	1    5075 4200
 	1    0    0    -1
@@
 F 2 "Connector_PinHeader_2.54mm:PinHeader_1x03_P2.54mm_Vertical" H 7350 3225 50  0001 C CNN
 F 3 "~" H 7350 3225 50  0001 C CNN
+F 4 "C376076" H 7350 3225 50  0001 C CNN "LCSC"
 	1    7350 3225
 	1    0    0    -1
@@
 L B.B-rescue:GND-B.B-eagle-import #GND0152
 U 1 1 60BC8FEF
-P 7050 4550
-F 0 "#GND0152" H 7050 4550 50  0001 C CNN
-F 1 "GND-B.B-eagle-import" H 7050 4470 59  0000 C CNN
-F 2 "" H 7050 4550 50  0001 C CNN
-F 3 "" H 7050 4550 50  0001 C CNN
-	1    7050 4550
+P 7050 4450
+F 0 "#GND0152" H 7050 4450 50  0001 C CNN
+F 1 "GND-B.B-eagle-import" H 7050 4370 59  0000 C CNN
+F 2 "" H 7050 4450 50  0001 C CNN
+F 3 "" H 7050 4450 50  0001 C CNN
+	1    7050 4450
 	1    0    0    -1
 $EndComp
@@
 	7100 3125 7100 3450
 Wire Wire Line
-	7050 3325 7150 3325
-Wire Wire Line
-	7150 3650 7050 3650
-Wire Wire Line
-	7050 3325 7050 3650
-Connection ~ 7050 3650
-Wire Wire Line
-	7050 3650 7050 3975
-Wire Wire Line
-	7050 3975 7150 3975
-Connection ~ 7050 3975
-Wire Wire Line
-	7150 4300 7050 4300
-Wire Wire Line
-	7050 3975 7050 4300
-Connection ~ 7050 4300
-Wire Wire Line
-	7050 4300 7050 4450
+	7050 3225 7150 3225
+Wire Wire Line
+	7150 3550 7050 3550
+Wire Wire Line
+	7050 3225 7050 3550
+Connection ~ 7050 3550
+Wire Wire Line
+	7050 3550 7050 3875
+Wire Wire Line
+	7050 3875 7150 3875
+Connection ~ 7050 3875
+Wire Wire Line
+	7150 4200 7050 4200
+Wire Wire Line
+	7050 3875 7050 4200
+Connection ~ 7050 4200
+Wire Wire Line
+	7050 4200 7050 4350
 $Comp
 L Connector_Generic:Conn_01x03 J11
@@
 F 2 "Connector_PinHeader_2.54mm:PinHeader_1x03_P2.54mm_Vertical" H 7350 3550 50  0001 C CNN
 F 3 "~" H 7350 3550 50  0001 C CNN
+F 4 "C376076" H 7350 3550 50  0001 C CNN "LCSC"
 	1    7350 3550
 	1    0    0    -1
@@
 F 2 "Connector_PinHeader_2.54mm:PinHeader_1x03_P2.54mm_Vertical" H 7350 3875 50  0001 C CNN
 F 3 "~" H 7350 3875 50  0001 C CNN
+F 4 "C376076" H 7350 3875 50  0001 C CNN "LCSC"
 	1    7350 3875
 	1    0    0    -1
@@
 F 2 "Connector_PinHeader_2.54mm:PinHeader_1x03_P2.54mm_Vertical" H 7350 4200 50  0001 C CNN
 F 3 "~" H 7350 4200 50  0001 C CNN
+F 4 "C376076" H 7350 4200 50  0001 C CNN "LCSC"
 	1    7350 4200
 	1    0    0    -1
 $EndComp
-Text HLabel 6975 3225 0    50   Input ~ 0
+Text HLabel 6975 3325 0    50   Input ~ 0
 T0
 Wire Wire Line
-	6975 3225 7150 3225
-Text HLabel 6975 3550 0    50   Input ~ 0
+	6975 3325 7150 3325
+Text HLabel 6975 3650 0    50   Input ~ 0
 T1
 Wire Wire Line
-	6975 3550 7150 3550
-Text HLabel 6975 3875 0    50   Input ~ 0
+	6975 3650 7150 3650
+Text HLabel 6975 3975 0    50   Input ~ 0
 T2
 Wire Wire Line
-	6975 3875 7150 3875
-Text HLabel 6975 4200 0    50   Input ~ 0
+	6975 3975 7150 3975
+Text HLabel 6975 4300 0    50   Input ~ 0
 T3
 Wire Wire Line
-	6975 4200 7150 4200
+	6975 4300 7150 4300
 Text Notes 7100 2650 0    50   ~ 0
 Tlacitka

Commit message: presuny_konektoru
Parts:
- added R12, R17, R39, R40: 12k, Resistor_SMD:R_0402_1005Metric, symbol B.B-rescue:R-Device-B.B-rescue
Connections:
- net 3.3V: now also R12.1, R17.1, R39.1, R40.1
- net T0: now also R12.2
- net T1: now also R17.2
- net T2: now also R39.2
- net T3: now also R40.2
Changed lines of the file:
@@
 $Descr A4 11693 8268
 encoding utf-8
-Sheet 8 9
+Sheet 7 9
 Title ""
 Date ""
@@
 	1    0    0    -1
 $EndComp
-Text HLabel 6975 3325 0    50   Input ~ 0
+Text HLabel 6775 3325 0    50   Input ~ 0
 T0
 Wire Wire Line
-	6975 3325 7150 3325
-Text HLabel 6975 3650 0    50   Input ~ 0
+	6775 3325 7000 3325
+Text HLabel 6750 3650 0    50   Input ~ 0
 T1
-Wire Wire Line
-	6975 3650 7150 3650
-Text HLabel 6975 3975 0    50   Input ~ 0
+Text HLabel 6750 3975 0    50   Input ~ 0
 T2
 Wire Wire Line
-	6975 3975 7150 3975
-Text HLabel 6975 4300 0    50   Input ~ 0
+	6750 3975 7000 3975
+Text HLabel 6750 4300 0    50   Input ~ 0
 T3
-Wire Wire Line
-	6975 4300 7150 4300
 Text Notes 7100 2650 0    50   ~ 0
 Tlacitka
@@
 Wire Notes Line
 	5750 2500 5750 4750
+$Comp
+L B.B-rescue:R-Device-B.B-rescue R?
+U 1 1 60A9DBE7
+P 6800 4225
+AR Path="/5F77B818/60A9DBE7" Ref="R?"  Part="1"
+AR Path="/60BC23E6/60A9DBE7" Ref="R40"  Part="1"
+F 0 "R40" V 6870 4271 50  0000 L CNN
+F 1 "12k" V 6875 4050 50  0000 L CNN
+F 2 "Resistor_SMD:R_0402_1005Metric" V 6730 4225 50  0001 C CNN
+F 3 "~" H 6800 4225 50  0001 C CNN
+F 4 "C25752" H 6800 4225 50  0001 C CNN "LCSC"
+	1    6800 4225
+	0    -1   -1   0
+$EndComp
+Wire Wire Line
+	6750 3650 7000 3650
+Wire Wire Line
+	6750 4300 7000 4300
+Wire Wire Line
+	6950 4225 7000 4225
+Wire Wire Line
+	7000 4225 7000 4300
+Connection ~ 7000 4300
+Wire Wire Line
+	7000 4300 7150 4300
+Wire Wire Line
+	6650 4225 6600 4225
+Wire Wire Line
+	6600 4225 6600 4100
+Wire Wire Line
+	6600 4100 7100 4100
+Connection ~ 7100 4100
+$Comp
+L B.B-rescue:R-Device-B.B-rescue R?
+U 1 1 60AB3CD2
+P 6800 3900
+AR Path="/5F77B818/60AB3CD2" Ref="R?"  Part="1"
+AR Path="/60BC23E6/60AB3CD2" Ref="R39"  Part="1"
+F 0 "R39" V 6870 3946 50  0000 L CNN
+F 1 "12k" V 6875 3725 50  0000 L CNN
+F 2 "Resistor_SMD:R_0402_1005Metric" V 6730 3900 50  0001 C CNN
+F 3 "~" H 6800 3900 50  0001 C CNN
+F 4 "C25752" H 6800 3900 50  0001 C CNN "LCSC"
+	1    6800 3900
+	0    -1   -1   0
+$EndComp
+Wire Wire Line
+	6950 3900 7000 3900
+Wire Wire Line
+	7000 3900 7000 3975
+Wire Wire Line
+	6650 3900 6600 3900
+Wire Wire Line
+	6600 3900 6600 3775
+Wire Wire Line
+	6600 3775 7100 3775
+$Comp
+L B.B-rescue:R-Device-B.B-rescue R?
+U 1 1 60AB5228
+P 6800 3575
+AR Path="/5F77B818/60AB5228" Ref="R?"  Part="1"
+AR Path="/60BC23E6/60AB5228" Ref="R17"  Part="1"
+F 0 "R17" V 6870 3621 50  0000 L CNN
+F 1 "12k" V 6875 3400 50  0000 L CNN
+F 2 "Resistor_SMD:R_0402_1005Metric" V 6730 3575 50  0001 C CNN
+F 3 "~" H 6800 3575 50  0001 C CNN
+F 4 "C25752" H 6800 3575 50  0001 C CNN "LCSC"
+	1    6800 3575
+	0    -1   -1   0
+$EndComp
+Wire Wire Line
+	6950 3575 7000 3575
+Wire Wire Line
+	7000 3575 7000 3650
+Wire Wire Line
+	6650 3575 6600 3575
+Wire Wire Line
+	6600 3575 6600 3450
+Wire Wire Line
+	6600 3450 7100 3450
+$Comp
+L B.B-rescue:R-Device-B.B-rescue R?
+U 1 1 60AB63BD
+P 6800 3250
+AR Path="/5F77B818/60AB63BD" Ref="R?"  Part="1"
+AR Path="/60BC23E6/60AB63BD" Ref="R12"  Part="1"
+F 0 "R12" V 6870 3296 50  0000 L CNN
+F 1 "12k" V 6875 3075 50  0000 L CNN
+F 2 "Resistor_SMD:R_0402_1005Metric" V 6730 3250 50  0001 C CNN
+F 3 "~" H 6800 3250 50  0001 C CNN
+F 4 "C25752" H 6800 3250 50  0001 C CNN "LCSC"
+	1    6800 3250
+	0    -1   -1   0
+$EndComp
+Wire Wire Line
+	6950 3250 7000 3250
+Wire Wire Line
+	7000 3250 7000 3325
+Wire Wire Line
+	6650 3250 6600 3250
+Wire Wire Line
+	6600 3250 6600 3125
+Wire Wire Line
+	6600 3125 7100 3125
+Connection ~ 7000 3325
+Wire Wire Line
+	7000 3325 7150 3325
+Connection ~ 7000 3650
+Wire Wire Line
+	7000 3650 7150 3650
+Connection ~ 7000 3975
+Wire Wire Line
+	7000 3975 7150 3975
 $EndSCHEMATC

Commit message: new schema
Parts:
- J10, J11, J12, J13, J14, J15, J8, J9: JLCPCB_CORRECTION (none) -> 0;2.54;90; LCSC C376076 -> C306138
Changed lines of the file:
@@
 EESchema Schematic File Version 4
-LIBS:B.B-cache
-EELAYER 29 0
+EELAYER 30 0
 EELAYER END
 $Descr A4 11693 8268
@@
 F 2 "Connector_PinHeader_2.54mm:PinHeader_1x03_P2.54mm_Vertical" H 5075 3225 50  0001 C CNN
 F 3 "~" H 5075 3225 50  0001 C CNN
-F 4 "C376076 " H 5075 3225 50  0001 C CNN "LCSC"
+F 4 "C306138" H 5075 3225 50  0001 C CNN "LCSC"
+F 5 "0;2.54;90" H 5075 3225 50  0001 C CNN "JLCPCB_CORRECTION"
 	1    5075 3225
 	1    0    0    -1
@@
 F 2 "Connector_PinHeader_2.54mm:PinHeader_1x03_P2.54mm_Vertical" H 5075 3550 50  0001 C CNN
 F 3 "~" H 5075 3550 50  0001 C CNN
-F 4 "C376076 " H 5075 3550 50  0001 C CNN "LCSC"
+F 4 "C306138" H 5075 3550 50  0001 C CNN "LCSC"
+F 5 "0;2.54;90" H 5075 3550 50  0001 C CNN "JLCPCB_CORRECTION"
 	1    5075 3550
 	1    0    0    -1
@@
 F 2 "Connector_PinHeader_2.54mm:PinHeader_1x03_P2.54mm_Vertical" H 5075 3875 50  0001 C CNN
 F 3 "~" H 5075 3875 50  0001 C CNN
-F 4 "C376076 " H 5075 3875 50  0001 C CNN "LCSC"
+F 4 "C306138" H 5075 3875 50  0001 C CNN "LCSC"
+F 5 "0;2.54;90" H 5075 3875 50  0001 C CNN "JLCPCB_CORRECTION"
 	1    5075 3875
 	1    0    0    -1
@@
 F 2 "Connector_PinHeader_2.54mm:PinHeader_1x03_P2.54mm_Vertical" H 5075 4200 50  0001 C CNN
 F 3 "~" H 5075 4200 50  0001 C CNN
-F 4 "C376076" H 5075 4200 50  0001 C CNN "LCSC"
+F 4 "C306138" H 5075 4200 50  0001 C CNN "LCSC"
+F 5 "0;2.54;90" H 5075 4200 50  0001 C CNN "JLCPCB_CORRECTION"
 	1    5075 4200
 	1    0    0    -1
@@
 F 2 "Connector_PinHeader_2.54mm:PinHeader_1x03_P2.54mm_Vertical" H 7350 3225 50  0001 C CNN
 F 3 "~" H 7350 3225 50  0001 C CNN
-F 4 "C376076" H 7350 3225 50  0001 C CNN "LCSC"
+F 4 "C306138" H 7350 3225 50  0001 C CNN "LCSC"
+F 5 "0;2.54;90" H 7350 3225 50  0001 C CNN "JLCPCB_CORRECTION"
 	1    7350 3225
 	1    0    0    -1
@@
 F 2 "Connector_PinHeader_2.54mm:PinHeader_1x03_P2.54mm_Vertical" H 7350 3550 50  0001 C CNN
 F 3 "~" H 7350 3550 50  0001 C CNN
-F 4 "C376076" H 7350 3550 50  0001 C CNN "LCSC"
+F 4 "C306138" H 7350 3550 50  0001 C CNN "LCSC"
+F 5 "0;2.54;90" H 7350 3550 50  0001 C CNN "JLCPCB_CORRECTION"
 	1    7350 3550
 	1    0    0    -1
@@
 F 2 "Connector_PinHeader_2.54mm:PinHeader_1x03_P2.54mm_Vertical" H 7350 3875 50  0001 C CNN
 F 3 "~" H 7350 3875 50  0001 C CNN
-F 4 "C376076" H 7350 3875 50  0001 C CNN "LCSC"
+F 4 "C306138" H 7350 3875 50  0001 C CNN "LCSC"
+F 5 "0;2.54;90" H 7350 3875 50  0001 C CNN "JLCPCB_CORRECTION"
 	1    7350 3875
 	1    0    0    -1
@@
 F 2 "Connector_PinHeader_2.54mm:PinHeader_1x03_P2.54mm_Vertical" H 7350 4200 50  0001 C CNN
 F 3 "~" H 7350 4200 50  0001 C CNN
-F 4 "C376076" H 7350 4200 50  0001 C CNN "LCSC"
+F 4 "C306138" H 7350 4200 50  0001 C CNN "LCSC"
+F 5 "0;2.54;90" H 7350 4200 50  0001 C CNN "JLCPCB_CORRECTION"
 	1    7350 4200
 	1    0    0    -1
