File: hw/RB3203/Charger.kicad_sch (KiCad schematic)
At the start: 18 parts

Commit message: Wip
Parts:
- U? (x3): value 0.1uf -> 0.1u
- U? (x4): value 22uf -> 22u
Changed lines of the file:
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@@
       (effects (font (size 1.27 1.27)) (justify left))
     )
-    (property "Value" "0.1uf" (id 1) (at 193.421 80.518 0)
+    (property "Value" "0.1u" (id 1) (at 193.421 80.518 0)
       (effects (font (size 1.27 1.27)) (justify left))
     )
@@
       (effects (font (size 1.27 1.27)) (justify left))
     )
-    (property "Value" "22uf" (id 1) (at 88.011 81.153 0)
+    (property "Value" "22u" (id 1) (at 88.011 81.153 0)
       (effects (font (size 1.27 1.27)) (justify left))
     )
@@
       (effects (font (size 1.27 1.27)) (justify left))
     )
-    (property "Value" "22uf" (id 1) (at 108.331 81.153 0)
+    (property "Value" "22u" (id 1) (at 108.331 81.153 0)
       (effects (font (size 1.27 1.27)) (justify left))
     )
@@
       (effects (font (size 1.27 1.27)) (justify left))
     )
-    (property "Value" "22uf" (id 1) (at 98.171 81.153 0)
+    (property "Value" "22u" (id 1) (at 98.171 81.153 0)
       (effects (font (size 1.27 1.27)) (justify left))
     )
@@
       (effects (font (size 1.27 1.27)) (justify left))
     )
-    (property "Value" "22uf" (id 1) (at 215.011 80.518 0)
+    (property "Value" "22u" (id 1) (at 215.011 80.518 0)
       (effects (font (size 1.27 1.27)) (justify left))
     )
@@
       (effects (font (size 1.27 1.27)) (justify left))
     )
-    (property "Value" "0.1uf" (id 1) (at 126.365 94.615 0)
+    (property "Value" "0.1u" (id 1) (at 126.365 94.615 0)
       (effects (font (size 1.27 1.27)) (justify left))
     )
@@
       (effects (font (size 1.27 1.27)) (justify left))
     )
-    (property "Value" "0.1uf" (id 1) (at 164.465 94.615 0)
-      (effects (font (size 1.27 1.27)) (justify left))
-    )
+    (property "Value" "0.1u" (id 1) (at 164.465 94.615 0)
+      (effects (font (size 1.27 1.27)) (justify left))
+    )
