File: hw/RB3203/ESPCircle.kicad_sch (KiCad schematic)
At the start: 54 parts

Commit message: Wip
Parts:
- removed ESP-?: ESP32-WROVER, RB3203-Lib:ESP32-WROVER, symbol RB3203-Lib:ESP32-WROVER
- removed U? (x20): NC, symbol B.B-rescue:NC-B.B-eagle-import-B.B-rescue
- removed U? (x5): 220, Resistor_SMD:R_0402_1005Metric, symbol B.B-rescue:R-Device-B.B-rescue-B.B-rescue
- removed U? (x2): SW_DIP_x01, Button_Switch_SMD:SW_Push_1P1T_NO_CK_KSC6xxJ, symbol B.B-rescue:SW_DIP_x01-Switch-B.B-rescue-B.B-rescue
- removed U? (x2): 0.1uf, Capacitor_SMD:C_0805_2012Metric, symbol B.B-rescue:C-Device-B.B-rescue-B.B-rescue
- removed U? (x2): 1M, Resistor_SMD:R_0402_1005Metric, symbol B.B-rescue:R-Device-B.B-rescue-B.B-rescue
- removed U? (x2): Q_NPN_BCE, Package_TO_SOT_SMD:SOT-23, symbol B.B-rescue:Q_NPN_BCE-B.B-rescue-B.B-rescue
- removed U? (x8): 12k, Resistor_SMD:R_0402_1005Metric, symbol B.B-rescue:R-Device-B.B-rescue-B.B-rescue
- removed U?: CP2102, Package_DFN_QFN:QFN-28-1EP_5x5mm_P0.5mm_EP3.35x3.35mm, symbol RB3203-Lib:CP2102
- removed U? (x2): 470, Resistor_SMD:R_0402_1005Metric, symbol B.B-rescue:R-Device-B.B-rescue-B.B-rescue
- removed U? (x2): RED, LED_SMD:LED_0603_1608Metric, symbol B.B-rescue:LED-B.B-eagle-import-B.B-rescue
- removed U? (x2): 100nf, Capacitor_SMD:C_0402_1005Metric, symbol B.B-rescue:C-Device-B.B-rescue-B.B-rescue
- removed U?: AO3400A, Package_TO_SOT_SMD:SOT-23, symbol B.B-rescue:2N7002-Transistor_FET-B.B-rescue-B.B-rescue
- removed U?: 1K, Resistor_SMD:R_0402_1005Metric, symbol B.B-rescue:R-Device-B.B-rescue-B.B-rescue
- removed U?: SW_DIP_x02, BB:SW-SMD-4, symbol B.B-rescue:SW_DIP_x02-Switch-B.B-rescue-B.B-rescue
- removed U? (x2): 10uf, Capacitor_SMD:C_0805_2012Metric, symbol B.B-rescue:C-Device-B.B-rescue-B.B-rescue
- added BOOT?, RESET?: button, my_library:Tactile_switch, symbol Switch:SW_Push
- added C?: 100n, Capacitor_SMD:C_0402_1005Metric, symbol Device:C
- added C? (x2): 1u, Capacitor_SMD:C_0402_1005Metric, symbol Device:C
- added C?: 10uF, Capacitor_SMD:C_0603_1608Metric, symbol Device:C
- added D? (x2): green, LED_SMD:LED_0603_1608Metric, symbol Device:LED
- added Q? (x2): Q_NPN_BEC, Package_TO_SOT_SMD:SOT-23, symbol Device:Q_NPN_BEC
- added R? (x10): 10k, Resistor_SMD:R_0402_1005Metric, symbol Device:R
- added SW?: SW_DIP_x01, symbol Switch:SW_DIP_x01
- added U?: 10uf, Capacitor_SMD:C_0805_2012Metric, symbol B.B-rescue:C-Device-B.B-rescue-B.B-rescue
- added U? (x2): 1M, Resistor_SMD:R_0402_1005Metric, symbol B.B-rescue:R-Device-B.B-rescue-B.B-rescue
- added U?: ESP32-S3-WROOM, Robotarna_KiCad_Library:ESP32-S3-WROOM, symbol Robotarna_KiCad_Library:ESP32-S3-WROOM
- added U?: CP2102N-A01-GQFN28, Package_DFN_QFN:QFN-28-1EP_5x5mm_P0.5mm_EP3.35x3.35mm, symbol Logic_tabor-rescue:CP2102N-A01-GQFN28-Interface_USB
- added U?: 220, Resistor_SMD:R_0402_1005Metric, symbol B.B-rescue:R-Device-B.B-rescue-B.B-rescue
- added U?: 0.1uf, Capacitor_SMD:C_0805_2012Metric, symbol B.B-rescue:C-Device-B.B-rescue-B.B-rescue
- added U?: AO3400A, Package_TO_SOT_SMD:SOT-23, symbol B.B-rescue:2N7002-Transistor_FET-B.B-rescue-B.B-rescue
Connections:
- net 3V3: now also C?.2, C?.2, R?.1, R?.1, U?.2 (3V3), U?.3 (D)
- net EN: now also C?.1, Q?.3 (C), R?.2, RESET?.1, U?.3 (EN)
- net GND: now also BOOT?.2, C?.1, C?.1, C?.2, C?.2, R?.2, R?.2, R?.2, RESET?.2, U?.1 (GND), U?.2, U?.2, U?.2, U?.2, U?.29 (GND), U?.3 (GND), U?.40 (GND), U?.41 (GND)
- net IO13: now also U?.21 (IO13)
- net IO14: now also U?.22 (IO14)
- net IO18: now also U?.11 (IO18)
- net IO21: now also U?.23 (IO21)
- net IO35: now also U?.28 (IO35)
- net IO39: now also U?.32 (IO39)
- net cabel_power-1.5-12V: now also SW?.1
- net cable_connected: now also R?.1, U?.1, U?.16 (IO46-PD)
- new net: D?.1 (K), R?.1 (x2)
- new net: D?.2 (A), D?.2 (A), R?.1, U?.1, U?.1, U?.1, U?.2, U?.2 (S), U?.6 (VDD), U?.7 (REGIN), U?.8 (VBUS)
- new net: Q?.1 (B), R?.1 (x2)
- new net: Q?.2 (E), R?.2, U?.24 (~{RTS})
- new net: Q?.2 (E), R?.2, U?.28 (~{DTR})
- new net: R?.2, U?.18 (~{RXT}/GPIO.1)
- new net: R?.2, U?.19 (~{TXT}/GPIO.0)
- new net: R?.2, U?.9 (~{RSTb})
- new net: SW?.2, U?.1, U?.1 (G)
- new net D+_ESP: U?.14 (IO20-D+)
- new net D+_UART: U?.4 (D+)
- new net D-_ESP: U?.13 (IO19-D-)
- new net D-_UART: U?.5 (D-)
- new net IO00-PU: BOOT?.1, C?.1, Q?.3 (C), R?.2, U?.27 (IO00-PU)
- new net IO01: U?.39 (IO01)
- new net IO02: U?.38 (IO02)
- new net IO03-PD: R?.1, U?.15 (IO03-PD)
- new net IO04: U?.4 (IO04)
- new net IO05: U?.5 (IO05)
- new net IO06: U?.6 (IO06)
- new net IO07: U?.7 (IO07)
- new net IO08: U?.12 (IO08)
- new net IO09: U?.17 (IO09)
- new net IO10: U?.18 (IO10)
- new net IO11: U?.19 (IO11)
- new net IO12: U?.20 (IO12)
- new net IO15: U?.8 (IO15)
- new net IO16: U?.9 (IO16)
- new net IO17: U?.10 (IO17)
- new net IO36: U?.29 (IO36)
- new net IO37: U?.30 (IO37)
- new net IO38: U?.31 (IO38)
- new net IO40: U?.33 (IO40)
- new net IO41: U?.34 (IO41)
- new net IO42: U?.35 (IO42)
- new net IO45-PD: R?.1, U?.26 (IO45-PD)
- new net IO47: U?.24 (IO47)
- new net IO48: U?.25 (IO48)
- new net RX_ESP: U?.26 (TXD), U?.36 (IO44-RX)
- new net TX_ESP: U?.25 (RXD), U?.37 (IO43-TX)
- no-connect marks 0 -> 14

Commit message: Wip
Parts:
- added U?: 1M, Resistor_SMD:R_0402_1005Metric, symbol B.B-rescue:R-Device-B.B-rescue-B.B-rescue
Connections:
- net GND: now also U?.2; no longer U?.2
- net cable_connected: now also D?.2 (A), D?.2 (A), R?.1, U?.1, U?.1, U?.1, U?.2, U?.2 (S), U?.6 (VDD), U?.7 (REGIN), U?.8 (VBUS)
- net at SW?.2, U?.1: no longer U?.1 (G)
- net cabel_power-1.5-12V renamed VUSB
- new net: U?.1, U?.1 (G), U?.2
Other:
- note added: "ESP32S3"
- note added: "Power saver"
- note added: "Programer"
- note added: "straping pins boot definition"
- moved on the sheet: D?, Q?, R?, SW?, U?

Commit message: Wip
Parts:
- C?: value 10uF -> 10u
- U?: value 0.1uf -> 0.1u
Changed lines of the file:
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@@
     (in_bom yes) (on_board yes)
     (property "Reference" "C?" (id 0) (at 246.38 30.48 90))
-    (property "Value" "10uF" (id 1) (at 254 30.48 90))
+    (property "Value" "10u" (id 1) (at 254 30.48 90))
     (property "Footprint" "Capacitor_SMD:C_0603_1608Metric" (id 2) (at 246.38 32.7152 0)
       (effects (font (size 1.27 1.27)) hide)
@@
       (effects (font (size 1.27 1.27)) (justify left))
     )
-    (property "Value" "0.1uf" (id 1) (at 80.01 63.5 0)
+    (property "Value" "0.1u" (id 1) (at 80.01 63.5 0)
       (effects (font (size 1.27 1.27)) (justify left))
     )
