File: hw/RB3203/ServoBoard.kicad_sch (KiCad schematic)
At the start: 7 parts

Commit message: Wip
Parts:
- C?: value 1uf -> 1u
- C?: value 0.1uf -> 0.1u
Changed lines of the file:
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@@
     (in_bom yes) (on_board yes)
     (property "Reference" "C?" (id 0) (at 110.49 65.405 0))
-    (property "Value" "1uf" (id 1) (at 110.49 70.485 0))
+    (property "Value" "1u" (id 1) (at 110.49 70.485 0))
     (property "Footprint" "Capacitor_SMD:C_0402_1005Metric" (id 2) (at 106.9848 64.135 0)
       (effects (font (size 1.27 1.27)) hide)
@@
       (effects (font (size 1.27 1.27)) (justify left))
     )
-    (property "Value" "0.1uf" (id 1) (at 101.6 70.485 0)
+    (property "Value" "0.1u" (id 1) (at 101.6 70.485 0)
       (effects (font (size 1.27 1.27)) (justify left))
     )
