File: hw/RB3203/USB.kicad_sch (KiCad schematic)
At the start: 25 parts

Commit message: Wip
Parts:
- C? (x3): value 100nF -> 100n
- C? (x2): value 1uF -> 1u
- C?: value 10uF -> 10u
- R? (x2): value 4k7 -> 4.7k
- R? (x2): value 5k1 -> 5.1k
Changed lines of the file:
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@@
     (in_bom yes) (on_board yes)
     (property "Reference" "C?" (id 0) (at 170.18 49.53 90))
-    (property "Value" "100nF" (id 1) (at 171.45 52.07 90))
+    (property "Value" "100n" (id 1) (at 171.45 52.07 90))
     (property "Footprint" "Capacitor_SMD:C_0402_1005Metric" (id 2) (at 175.26 54.9148 0)
       (effects (font (size 1.27 1.27)) hide)
@@
       (effects (font (size 1.27 1.27)) (justify left))
     )
-    (property "Value" "1uF" (id 1) (at 163.83 93.98 0)
+    (property "Value" "1u" (id 1) (at 163.83 93.98 0)
       (effects (font (size 1.27 1.27)) (justify left))
     )
@@
       (effects (font (size 1.27 1.27)) (justify left))
     )
-    (property "Value" "10uF" (id 1) (at 140.97 50.8 0)
+    (property "Value" "10u" (id 1) (at 140.97 50.8 0)
       (effects (font (size 1.27 1.27)) (justify left))
     )
@@
       (effects (font (size 1.27 1.27)) (justify left))
     )
-    (property "Value" "4k7" (id 1) (at 223.52 88.9 90)
+    (property "Value" "4.7k" (id 1) (at 223.52 88.9 90)
       (effects (font (size 1.27 1.27)) (justify left))
     )
@@
       (effects (font (size 1.27 1.27)) (justify left))
     )
-    (property "Value" "1uF" (id 1) (at 220.98 55.8799 0)
+    (property "Value" "1u" (id 1) (at 220.98 55.8799 0)
       (effects (font (size 1.27 1.27)) (justify left))
     )
@@
     (in_bom yes) (on_board yes)
     (property "Reference" "R?" (id 0) (at 85.09 128.27 90))
-    (property "Value" "5k1" (id 1) (at 90.17 128.27 90))
+    (property "Value" "5.1k" (id 1) (at 90.17 128.27 90))
     (property "Footprint" "Resistor_SMD:R_0402_1005Metric" (id 2) (at 86.36 123.952 90)
       (effects (font (size 1.27 1.27)) hide)
@@
     (in_bom yes) (on_board yes)
     (property "Reference" "C?" (id 0) (at 213.36 91.44 0))
-    (property "Value" "100nF" (id 1) (at 214.63 93.98 0))
+    (property "Value" "100n" (id 1) (at 214.63 93.98 0))
     (property "Footprint" "Capacitor_SMD:C_0402_1005Metric" (id 2) (at 207.3148 88.9 0)
       (effects (font (size 1.27 1.27)) hide)
@@
       (effects (font (size 1.27 1.27)) (justify left))
     )
-    (property "Value" "4k7" (id 1) (at 149.86 52.07 90)
+    (property "Value" "4.7k" (id 1) (at 149.86 52.07 90)
       (effects (font (size 1.27 1.27)) (justify left))
     )
@@
     (in_bom yes) (on_board yes)
     (property "Reference" "R?" (id 0) (at 85.09 120.65 90))
-    (property "Value" "5k1" (id 1) (at 90.17 120.65 90))
+    (property "Value" "5.1k" (id 1) (at 90.17 120.65 90))
     (property "Footprint" "Resistor_SMD:R_0402_1005Metric" (id 2) (at 86.36 121.412 90)
       (effects (font (size 1.27 1.27)) hide)
@@
     (in_bom yes) (on_board yes)
     (property "Reference" "C?" (id 0) (at 182.88 91.44 0))
-    (property "Value" "100nF" (id 1) (at 184.15 93.98 0))
+    (property "Value" "100n" (id 1) (at 184.15 93.98 0))
     (property "Footprint" "Capacitor_SMD:C_0402_1005Metric" (id 2) (at 176.8348 88.9 0)
       (effects (font (size 1.27 1.27)) hide)
