File: hw/RB3203/LedBoard.kicad_sch (KiCad schematic)
At the start: 22 parts

Commit message: Wip
Parts:
- C? (x2): value 10uf -> 10u
- C? (x2): value 1uf -> 1u
- C? (x3): value 10nf -> 10n
- C? (x2): value 0.1uf -> 0.1u
- C? (x4): value 1000pf -> 1000p
- C? (x2): value 100pf -> 100p
Changed lines of the file:
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@@
       (effects (font (size 1.27 1.27)) (justify left))
     )
-    (property "Value" "10uf" (id 1) (at 78.486 59.563 0)
+    (property "Value" "10u" (id 1) (at 78.486 59.563 0)
       (effects (font (size 1.27 1.27)) (justify left))
     )
@@
     (in_bom yes) (on_board yes)
     (property "Reference" "C?" (id 0) (at 184.912 83.058 0))
-    (property "Value" "1uf" (id 1) (at 184.912 88.138 0))
+    (property "Value" "1u" (id 1) (at 184.912 88.138 0))
     (property "Footprint" "Capacitor_SMD:C_0402_1005Metric" (id 2) (at 181.4068 81.788 0)
       (effects (font (size 1.27 1.27)) hide)
@@
       (effects (font (size 1.27 1.27)) (justify left))
     )
-    (property "Value" "10nf" (id 1) (at 196.215 88.138 0)
+    (property "Value" "10n" (id 1) (at 196.215 88.138 0)
       (effects (font (size 1.27 1.27)) (justify left))
     )
@@
       (effects (font (size 1.27 1.27)) (justify left))
     )
-    (property "Value" "10uf" (id 1) (at 89.281 59.563 0)
+    (property "Value" "10u" (id 1) (at 89.281 59.563 0)
       (effects (font (size 1.27 1.27)) (justify left))
     )
@@
       (effects (font (size 1.27 1.27)) (justify left))
     )
-    (property "Value" "0.1uf" (id 1) (at 67.056 107.696 0)
+    (property "Value" "0.1u" (id 1) (at 67.056 107.696 0)
       (effects (font (size 1.27 1.27)) (justify left))
     )
@@
     (in_bom yes) (on_board yes)
     (property "Reference" "C?" (id 0) (at 75.819 102.616 0))
-    (property "Value" "1uf" (id 1) (at 75.819 107.696 0))
+    (property "Value" "1u" (id 1) (at 75.819 107.696 0))
     (property "Footprint" "Capacitor_SMD:C_0402_1005Metric" (id 2) (at 72.3138 101.346 0)
       (effects (font (size 1.27 1.27)) hide)
@@
     (in_bom yes) (on_board yes)
     (property "Reference" "C?" (id 0) (at 136.652 120.396 90))
-    (property "Value" "1000pf" (id 1) (at 144.907 120.396 90))
+    (property "Value" "1000p" (id 1) (at 144.907 120.396 90))
     (property "Footprint" "Capacitor_SMD:C_0402_1005Metric" (id 2) (at 136.652 122.6312 0)
       (effects (font (size 1.27 1.27)) hide)
@@
       (effects (font (size 1.27 1.27)) (justify left))
     )
-    (property "Value" "10nf" (id 1) (at 60.452 107.696 0)
+    (property "Value" "10n" (id 1) (at 60.452 107.696 0)
       (effects (font (size 1.27 1.27)) (justify left))
     )
@@
     (in_bom yes) (on_board yes)
     (property "Reference" "C?" (id 0) (at 136.652 112.776 90))
-    (property "Value" "1000pf" (id 1) (at 144.907 112.776 90))
+    (property "Value" "1000p" (id 1) (at 144.907 112.776 90))
     (property "Footprint" "Capacitor_SMD:C_0402_1005Metric" (id 2) (at 136.652 115.0112 0)
       (effects (font (size 1.27 1.27)) hide)
@@
       (effects (font (size 1.27 1.27)) (justify left))
     )
-    (property "Value" "10nf" (id 1) (at 53.721 107.696 0)
+    (property "Value" "10n" (id 1) (at 53.721 107.696 0)
       (effects (font (size 1.27 1.27)) (justify left))
     )
@@
       (effects (font (size 1.27 1.27)) (justify left))
     )
-    (property "Value" "0.1uf" (id 1) (at 189.611 88.138 0)
+    (property "Value" "0.1u" (id 1) (at 189.611 88.138 0)
       (effects (font (size 1.27 1.27)) (justify left))
     )
@@
       (effects (font (size 1.27 1.27)) (justify left))
     )
-    (property "Value" "100pf" (id 1) (at 80.899 107.696 0)
+    (property "Value" "100p" (id 1) (at 80.899 107.696 0)
       (effects (font (size 1.27 1.27)) (justify left))
     )
@@
     (in_bom yes) (on_board yes)
     (property "Reference" "C?" (id 0) (at 136.652 105.156 90))
-    (property "Value" "1000pf" (id 1) (at 144.907 105.156 90))
+    (property "Value" "1000p" (id 1) (at 144.907 105.156 90))
     (property "Footprint" "Capacitor_SMD:C_0402_1005Metric" (id 2) (at 136.652 107.3912 0)
       (effects (font (size 1.27 1.27)) hide)
@@
     (in_bom yes) (on_board yes)
     (property "Reference" "C?" (id 0) (at 136.652 128.016 90))
-    (property "Value" "1000pf" (id 1) (at 144.907 128.016 90))
+    (property "Value" "1000p" (id 1) (at 144.907 128.016 90))
     (property "Footprint" "Capacitor_SMD:C_0402_1005Metric" (id 2) (at 136.652 130.2512 0)
       (effects (font (size 1.27 1.27)) hide)
@@
       (effects (font (size 1.27 1.27)) (justify left))
     )
-    (property "Value" "100pf" (id 1) (at 203.327 88.138 0)
-      (effects (font (size 1.27 1.27)) (justify left))
-    )
+    (property "Value" "100p" (id 1) (at 203.327 88.138 0)
+      (effects (font (size 1.27 1.27)) (justify left))
+    )

Commit message: Wip
Parts:
- removed C?: 1u, Capacitor_SMD:C_0402_1005Metric, symbol B.B-rescue:C-Device-B.B-rescue
- removed C?: 10n, Capacitor_SMD:C_0402_1005Metric, symbol B.B-rescue:C-Device-B.B-rescue
- removed C?: 0.1u, Resistor_SMD:R_0402_1005Metric, symbol B.B-rescue:C-Device-B.B-rescue
- removed C?: 100p, Capacitor_SMD:C_0402_1005Metric, symbol B.B-rescue:C-Device-B.B-rescue
- removed NFC?: M24SR64, symbol RB3203-Lib:M24SR64
Connections:
- net SHUTDOWN-LDC is gone; now on net AN-GND: U?.6 (SD)
Other:
- moved on the sheet: C?, J?, L?, U?
