File: hw/RB3203/MainBoard.kicad_sch (KiCad schematic)
At the start: 8 parts

Commit message: Wip
Parts:
- removed J?: Conn_01x04, symbol Connector_Generic:Conn_01x04
- removed J?: Conn_01x02, symbol Connector_Generic:Conn_01x02
- removed U? (x2): 100k, Resistor_SMD:R_0402_1005Metric, symbol B.B-rescue:R-Device-B.B-rescue-B.B-rescue
Other:
- sheet BatteriManager renamed PowerManager
- removed sheet A9G
- added sheet USB (USB.kicad_sch)
- sheet ESPCircle ports: added D+_ESP, D+_UART, D-_ESP, D-_UART, EN, IO00-PU, IO01, IO02, IO03-PD, IO04, IO05, IO06, IO07, IO08, IO09, IO10, IO11, IO12, IO15, IO16, IO17, IO36, IO37, IO38, IO40, IO41, IO42, IO45-PD, IO47, IO48; removed D+, D-, IO0-up, IO12-down, IO15-up, IO19, IO2-down, IO22, IO23, IO25, IO26, IO27, IO32, IO33, IO34, IO4, IO5-up
- sheet PowerManager: file BatteriManager.kicad_sch -> PowerManager.kicad_sch
- sheet PowerManager ports: added BUTTON_ON, EN, VCC; removed 4V, BATERIMETR, SHUTDOWN_3V3-5V
- moved on the sheet: U?

Commit message: Wip
Other:
- moved on the sheet: U?
Changed lines of the file:
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@@
   (junction (at 104.14 71.12) (diameter 0) (color 0 0 0 0)
   )
-  (junction (at 200.66 48.26) (diameter 0) (color 0 0 0 0)
+  (junction (at 118.11 96.52) (diameter 0) (color 0 0 0 0)
   )
   (junction (at 71.12 99.06) (diameter 0) (color 0 0 0 0)
   )
-  (junction (at 195.58 45.72) (diameter 0) (color 0 0 0 0)
+  (junction (at 118.11 45.72) (diameter 0) (color 0 0 0 0)
   )
   (junction (at 200.66 87.63) (diameter 0) (color 0 0 0 0)
   )
+  (junction (at 123.19 99.06) (diameter 0) (color 0 0 0 0)
+  )
   (junction (at 123.19 45.72) (diameter 0) (color 0 0 0 0)
   )
-  (wire (pts (xy 190.5 45.72) (xy 195.58 45.72))
+  (junction (at 118.11 101.6) (diameter 0) (color 0 0 0 0)
+  )
+  (junction (at 123.19 93.98) (diameter 0) (color 0 0 0 0)
+  )
+  (wire (pts (xy 118.11 45.72) (xy 123.19 45.72))
+    (stroke (width 0) (type default) (color 0 0 0 0))
+  )
+  (wire (pts (xy 101.6 96.52) (xy 118.11 96.52))
+    (stroke (width 0) (type default) (color 0 0 0 0))
+  )
+  (wire (pts (xy 127 99.06) (xy 123.19 99.06))
+    (stroke (width 0) (type default) (color 0 0 0 0))
+  )
+  (wire (pts (xy 101.6 45.72) (xy 118.11 45.72))
     (stroke (width 0) (type default) (color 0 0 0 0))
   )
@@
     (stroke (width 0) (type default) (color 0 0 0 0))
   )
+  (wire (pts (xy 114.3 101.6) (xy 118.11 101.6))
+    (stroke (width 0) (type default) (color 0 0 0 0))
+  )
   (wire (pts (xy 101.6 83.82) (xy 127 83.82))
     (stroke (width 0) (type default) (color 0 0 0 0))
@@
     (stroke (width 0) (type default) (color 0 0 0 0))
   )
-  (wire (pts (xy 190.5 48.26) (xy 200.66 48.26))
+  (wire (pts (xy 127 101.6) (xy 118.11 101.6))
     (stroke (width 0) (type default) (color 0 0 0 0))
   )
@@
     (stroke (width 0) (type default) (color 0 0 0 0))
   )
+  (wire (pts (xy 101.6 91.44) (xy 127 91.44))
+    (stroke (width 0) (type default) (color 0 0 0 0))
+  )
+  (wire (pts (xy 118.11 68.58) (xy 118.11 96.52))
+    (stroke (width 0) (type default) (color 0 0 0 0))
+  )
   (wire (pts (xy 190.5 87.63) (xy 200.66 87.63))
     (stroke (width 0) (type default) (color 0 0 0 0))
@@
     (stroke (width 0) (type default) (color 0 0 0 0))
   )
+  (wire (pts (xy 123.19 93.98) (xy 123.19 99.06))
+    (stroke (width 0) (type default) (color 0 0 0 0))
+  )
+  (wire (pts (xy 123.19 68.58) (xy 123.19 93.98))
+    (stroke (width 0) (type default) (color 0 0 0 0))
+  )
+  (wire (pts (xy 101.6 93.98) (xy 123.19 93.98))
+    (stroke (width 0) (type default) (color 0 0 0 0))
+  )
   (wire (pts (xy 200.66 87.63) (xy 203.2 87.63))
     (stroke (width 0) (type default) (color 0 0 0 0))
   )
-  (wire (pts (xy 200.66 43.18) (xy 200.66 48.26))
-    (stroke (width 0) (type default) (color 0 0 0 0))
-  )
   (wire (pts (xy 101.6 40.64) (xy 115.57 40.64))
     (stroke (width 0) (type default) (color 0 0 0 0))
@@
     (stroke (width 0) (type default) (color 0 0 0 0))
   )
-  (wire (pts (xy 200.66 48.26) (xy 203.2 48.26))
-    (stroke (width 0) (type default) (color 0 0 0 0))
-  )
   (wire (pts (xy 104.14 71.12) (xy 127 71.12))
     (stroke (width 0) (type default) (color 0 0 0 0))
@@
     (stroke (width 0) (type default) (color 0 0 0 0))
   )
-  (wire (pts (xy 101.6 45.72) (xy 123.19 45.72))
+  (wire (pts (xy 114.3 99.06) (xy 123.19 99.06))
+    (stroke (width 0) (type default) (color 0 0 0 0))
+  )
+  (wire (pts (xy 118.11 45.72) (xy 118.11 60.96))
     (stroke (width 0) (type default) (color 0 0 0 0))
   )
@@
     (stroke (width 0) (type default) (color 0 0 0 0))
   )
+  (wire (pts (xy 123.19 45.72) (xy 123.19 60.96))
+    (stroke (width 0) (type default) (color 0 0 0 0))
+  )
   (wire (pts (xy 190.5 60.96) (xy 203.2 60.96))
     (stroke (width 0) (type default) (color 0 0 0 0))
@@
     (stroke (width 0) (type default) (color 0 0 0 0))
   )
-  (wire (pts (xy 195.58 45.72) (xy 203.2 45.72))
+  (wire (pts (xy 118.11 96.52) (xy 118.11 101.6))
     (stroke (width 0) (type default) (color 0 0 0 0))
   )
   (wire (pts (xy 71.12 104.14) (xy 71.12 99.06))
-    (stroke (width 0) (type default) (color 0 0 0 0))
-  )
-  (wire (pts (xy 195.58 43.18) (xy 195.58 45.72))
     (stroke (width 0) (type default) (color 0 0 0 0))
   )
@@
     (effects (font (size 1.27 1.27)) (justify left))
   )
-  (hierarchical_label "SDA" (shape bidirectional) (at 203.2 45.72 0)
-    (effects (font (size 1.27 1.27)) (justify left))
+  (hierarchical_label "SDA" (shape bidirectional) (at 114.3 99.06 180)
+    (effects (font (size 1.27 1.27)) (justify right))
   )
   (hierarchical_label "GND" (shape output) (at 71.12 104.14 270)
@@
     (effects (font (size 1.27 1.27)) (justify left))
   )
-  (hierarchical_label "3V3" (shape output) (at 200.66 35.56 90)
-    (effects (font (size 1.27 1.27)) (justify left))
-  )
   (hierarchical_label "XRES" (shape output) (at 203.2 92.71 0)
     (effects (font (size 1.27 1.27)) (justify left))
   )
-  (hierarchical_label "SCL" (shape output) (at 203.2 48.26 0)
-    (effects (font (size 1.27 1.27)) (justify left))
+  (hierarchical_label "SCL" (shape output) (at 114.3 101.6 180)
+    (effects (font (size 1.27 1.27)) (justify right))
   )
   (hierarchical_label "3V3" (shape output) (at 200.66 74.93 90)
@@
     (effects (font (size 1.27 1.27)) (justify left))
   )
-  (hierarchical_label "3V3" (shape output) (at 195.58 35.56 90)
-    (effects (font (size 1.27 1.27)) (justify left))
-  )
   (hierarchical_label "INT-LDC" (shape output) (at 203.2 58.42 0)
     (effects (font (size 1.27 1.27)) (justify left))
   )
-  (symbol (lib_id "B.B-rescue:R-Device-B.B-rescue") (at 195.58 39.37 180) (unit 1)
+  (symbol (lib_id "B.B-rescue:R-Device-B.B-rescue") (at 123.19 64.77 0) (mirror x) (unit 1)
     (in_bom yes) (on_board yes)
-    (property "Reference" "U?" (id 0) (at 193.04 36.83 90))
-    (property "Value" "7.5k" (id 1) (at 193.04 41.91 90))
-    (property "Footprint" "Resistor_SMD:R_0402_1005Metric" (id 2) (at 197.358 39.37 90)
-      (effects (font (size 1.27 1.27)) hide)
-    )
-    (property "Datasheet" "~" (id 3) (at 195.58 39.37 0)
-      (effects (font (size 1.27 1.27)) hide)
-    )
-    (property "LCSC" "C25918" (id 4) (at 195.58 39.37 0)
+    (property "Reference" "U?" (id 0) (at 120.65 62.23 90))
+    (property "Value" "7.5k" (id 1) (at 120.65 67.31 90))
+    (property "Footprint" "Resistor_SMD:R_0402_1005Metric" (id 2) (at 121.412 64.77 90)
+      (effects (font (size 1.27 1.27)) hide)
+    )
+    (property "Datasheet" "~" (id 3) (at 123.19 64.77 0)
+      (effects (font (size 1.27 1.27)) hide)
+    )
+    (property "LCSC" "C25918" (id 4) (at 123.19 64.77 0)
       (effects (font (size 1.27 1.27)) hide)
     )
@@
     (pin "2")
   )
-  (symbol (lib_id "B.B-rescue:R-Device-B.B-rescue") (at 200.66 39.37 180) (unit 1)
+  (symbol (lib_id "B.B-rescue:R-Device-B.B-rescue") (at 118.11 64.77 0) (mirror x) (unit 1)
     (in_bom yes) (on_board yes)
-    (property "Reference" "U?" (id 0) (at 198.12 36.83 90))
-    (property "Value" "7.5k" (id 1) (at 198.12 41.91 90))
-    (property "Footprint" "Resistor_SMD:R_0402_1005Metric" (id 2) (at 202.438 39.37 90)
-      (effects (font (size 1.27 1.27)) hide)
-    )
-    (property "Datasheet" "~" (id 3) (at 200.66 39.37 0)
-      (effects (font (size 1.27 1.27)) hide)
-    )
-    (property "LCSC" "C25918" (id 4) (at 200.66 39.37 0)
+    (property "Reference" "U?" (id 0) (at 115.57 62.23 90))
+    (property "Value" "7.5k" (id 1) (at 115.57 67.31 90))
+    (property "Footprint" "Resistor_SMD:R_0402_1005Metric" (id 2) (at 116.332 64.77 90)
+      (effects (font (size 1.27 1.27)) hide)
+    )
+    (property "Datasheet" "~" (id 3) (at 118.11 64.77 0)
+      (effects (font (size 1.27 1.27)) hide)
+    )
+    (property "LCSC" "C25918" (id 4) (at 118.11 64.77 0)
       (effects (font (size 1.27 1.27)) hide)
     )
@@
       (effects (font (size 1.27 1.27)) (justify right))
     )
-    (pin "SCL" input (at 101.6 91.44 0)
+    (pin "SCL" input (at 101.6 96.52 0)
       (effects (font (size 1.27 1.27)) (justify right))
     )
@@
       (effects (font (size 1.27 1.27)) (justify right))
     )
-    (pin "INT" output (at 101.6 96.52 0)
+    (pin "INT" output (at 101.6 91.44 0)
       (effects (font (size 1.27 1.27)) (justify right))
     )
@@
       (effects (font (size 1.27 1.27)) (justify left))
     )
-    (pin "IO41" bidirectional (at 165.1 60.96 0)
-      (effects (font (size 1.27 1.27)) (justify right))
-    )
-    (pin "IO42" bidirectional (at 165.1 58.42 0)
-      (effects (font (size 1.27 1.27)) (justify right))
+    (pin "IO41" bidirectional (at 127 99.06 180)
+      (effects (font (size 1.27 1.27)) (justify left))
+    )
+    (pin "IO42" bidirectional (at 127 91.44 180)
+      (effects (font (size 1.27 1.27)) (justify left))
     )
     (pin "IO47" bidirectional (at 165.1 45.72 0)
       (effects (font (size 1.27 1.27)) (justify right))
     )
-    (pin "IO40" bidirectional (at 165.1 63.5 0)
-      (effects (font (size 1.27 1.27)) (justify right))
+    (pin "IO40" bidirectional (at 127 101.6 180)
+      (effects (font (size 1.27 1.27)) (justify left))
     )
     (pin "IO36" bidirectional (at 165.1 73.66 0)

Commit message: Wip
Parts:
- removed U? (x2): 7.5k, Resistor_SMD:R_0402_1005Metric, symbol B.B-rescue:R-Device-B.B-rescue
Other:
- added sheet LCB (LanternCommunicationBus.kicad_sch)
Changed lines of the file:
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@@
 (kicad_sch (version 20211123) (generator eeschema)
   (paper "A4")
-  (junction (at 195.58 85.09) (diameter 0) (color 0 0 0 0)
-  )
   (junction (at 104.14 71.12) (diameter 0) (color 0 0 0 0)
   )
@@
   (junction (at 118.11 45.72) (diameter 0) (color 0 0 0 0)
   )
-  (junction (at 200.66 87.63) (diameter 0) (color 0 0 0 0)
-  )
   (junction (at 123.19 99.06) (diameter 0) (color 0 0 0 0)
   )
@@
     (stroke (width 0) (type default) (color 0 0 0 0))
   )
-  (wire (pts (xy 195.58 82.55) (xy 195.58 85.09))
-    (stroke (width 0) (type default) (color 0 0 0 0))
-  )
-  (wire (pts (xy 190.5 58.42) (xy 203.2 58.42))
-    (stroke (width 0) (type default) (color 0 0 0 0))
-  )
-  (wire (pts (xy 190.5 53.34) (xy 203.2 53.34))
-    (stroke (width 0) (type default) (color 0 0 0 0))
-  )
-  (wire (pts (xy 190.5 92.71) (xy 203.2 92.71))
-    (stroke (width 0) (type default) (color 0 0 0 0))
-  )
   (wire (pts (xy 115.57 33.02) (xy 115.57 40.64))
     (stroke (width 0) (type default) (color 0 0 0 0))
@@
     (stroke (width 0) (type default) (color 0 0 0 0))
   )
-  (wire (pts (xy 190.5 85.09) (xy 195.58 85.09))
-    (stroke (width 0) (type default) (color 0 0 0 0))
-  )
   (wire (pts (xy 127 101.6) (xy 118.11 101.6))
     (stroke (width 0) (type default) (color 0 0 0 0))
@@
     (stroke (width 0) (type default) (color 0 0 0 0))
   )
-  (wire (pts (xy 190.5 90.17) (xy 203.2 90.17))
-    (stroke (width 0) (type default) (color 0 0 0 0))
-  )
   (wire (pts (xy 101.6 91.44) (xy 127 91.44))
     (stroke (width 0) (type default) (color 0 0 0 0))
@@
     (stroke (width 0) (type default) (color 0 0 0 0))
   )
-  (wire (pts (xy 190.5 87.63) (xy 200.66 87.63))
-    (stroke (width 0) (type default) (color 0 0 0 0))
-  )
   (wire (pts (xy 101.6 49.53) (xy 127 49.53))
     (stroke (width 0) (type default) (color 0 0 0 0))
@@
     (stroke (width 0) (type default) (color 0 0 0 0))
   )
-  (wire (pts (xy 200.66 87.63) (xy 203.2 87.63))
-    (stroke (width 0) (type default) (color 0 0 0 0))
-  )
   (wire (pts (xy 101.6 40.64) (xy 115.57 40.64))
     (stroke (width 0) (type default) (color 0 0 0 0))
@@
     (stroke (width 0) (type default) (color 0 0 0 0))
   )
-  (wire (pts (xy 190.5 60.96) (xy 203.2 60.96))
-    (stroke (width 0) (type default) (color 0 0 0 0))
-  )
   (wire (pts (xy 101.6 76.2) (xy 127 76.2))
     (stroke (width 0) (type default) (color 0 0 0 0))
@@
     (stroke (width 0) (type default) (color 0 0 0 0))
   )
-  (wire (pts (xy 190.5 66.04) (xy 203.2 66.04))
-    (stroke (width 0) (type default) (color 0 0 0 0))
-  )
   (wire (pts (xy 118.11 96.52) (xy 118.11 101.6))
     (stroke (width 0) (type default) (color 0 0 0 0))
@@
     (stroke (width 0) (type default) (color 0 0 0 0))
   )
-  (wire (pts (xy 190.5 55.88) (xy 203.2 55.88))
-    (stroke (width 0) (type default) (color 0 0 0 0))
-  )
   (wire (pts (xy 123.19 45.72) (xy 127 45.72))
     (stroke (width 0) (type default) (color 0 0 0 0))
   )
-  (wire (pts (xy 200.66 82.55) (xy 200.66 87.63))
-    (stroke (width 0) (type default) (color 0 0 0 0))
-  )
   (wire (pts (xy 123.19 35.56) (xy 123.19 45.72))
-    (stroke (width 0) (type default) (color 0 0 0 0))
-  )
-  (wire (pts (xy 195.58 85.09) (xy 203.2 85.09))
     (stroke (width 0) (type default) (color 0 0 0 0))
   )
@@
     (effects (font (size 1.27 1.27)) (justify right bottom))
   )
-  (hierarchical_label "SDA-2" (shape bidirectional) (at 203.2 85.09 0)
-    (effects (font (size 1.27 1.27)) (justify left))
-  )
   (hierarchical_label "SDA" (shape bidirectional) (at 114.3 99.06 180)
     (effects (font (size 1.27 1.27)) (justify right))
@@
     (effects (font (size 1.27 1.27)) (justify right))
   )
-  (hierarchical_label "INT-NFC" (shape output) (at 203.2 60.96 0)
-    (effects (font (size 1.27 1.27)) (justify left))
-  )
-  (hierarchical_label "3V3" (shape output) (at 195.58 74.93 90)
-    (effects (font (size 1.27 1.27)) (justify left))
-  )
-  (hierarchical_label "SHUTDOWN-NFC" (shape output) (at 203.2 55.88 0)
-    (effects (font (size 1.27 1.27)) (justify left))
-  )
   (hierarchical_label "3V3" (shape output) (at 123.19 35.56 90)
     (effects (font (size 1.27 1.27)) (justify left))
@@
     (effects (font (size 1.27 1.27)) (justify left))
   )
-  (hierarchical_label "INT-EXP" (shape input) (at 203.2 90.17 0)
-    (effects (font (size 1.27 1.27)) (justify left))
-  )
-  (hierarchical_label "SCL-2" (shape output) (at 203.2 87.63 0)
-    (effects (font (size 1.27 1.27)) (justify left))
-  )
-  (hierarchical_label "WS2812" (shape output) (at 203.2 66.04 0)
-    (effects (font (size 1.27 1.27)) (justify left))
-  )
-  (hierarchical_label "XRES" (shape output) (at 203.2 92.71 0)
-    (effects (font (size 1.27 1.27)) (justify left))
-  )
   (hierarchical_label "SCL" (shape output) (at 114.3 101.6 180)
     (effects (font (size 1.27 1.27)) (justify right))
-  )
-  (hierarchical_label "3V3" (shape output) (at 200.66 74.93 90)
-    (effects (font (size 1.27 1.27)) (justify left))
-  )
-  (hierarchical_label "SHUTDOWN-LDC" (shape output) (at 203.2 53.34 0)
-    (effects (font (size 1.27 1.27)) (justify left))
-  )
-  (hierarchical_label "INT-LDC" (shape output) (at 203.2 58.42 0)
-    (effects (font (size 1.27 1.27)) (justify left))
   )
   (symbol (lib_id "B.B-rescue:R-Device-B.B-rescue") (at 123.19 64.77 0) (mirror x) (unit 1)
@@
     (pin "2")
   )
-  (symbol (lib_id "B.B-rescue:R-Device-B.B-rescue") (at 200.66 78.74 180) (unit 1)
-    (in_bom yes) (on_board yes)
-    (property "Reference" "U?" (id 0) (at 198.12 76.2 90))
-    (property "Value" "7.5k" (id 1) (at 198.12 81.28 90))
-    (property "Footprint" "Resistor_SMD:R_0402_1005Metric" (id 2) (at 202.438 78.74 90)
-      (effects (font (size 1.27 1.27)) hide)
-    )
-    (property "Datasheet" "~" (id 3) (at 200.66 78.74 0)
-      (effects (font (size 1.27 1.27)) hide)
-    )
-    (property "LCSC" "C25918" (id 4) (at 200.66 78.74 0)
-      (effects (font (size 1.27 1.27)) hide)
-    )
-    (pin "1")
-    (pin "2")
-  )
   (symbol (lib_id "B.B-rescue:R-Device-B.B-rescue") (at 118.11 64.77 0) (mirror x) (unit 1)
     (in_bom yes) (on_board yes)
@@
     (pin "2")
   )
-  (symbol (lib_id "B.B-rescue:R-Device-B.B-rescue") (at 195.58 78.74 180) (unit 1)
-    (in_bom yes) (on_board yes)
-    (property "Reference" "U?" (id 0) (at 193.04 76.2 90))
-    (property "Value" "7.5k" (id 1) (at 193.04 81.28 90))
-    (property "Footprint" "Resistor_SMD:R_0402_1005Metric" (id 2) (at 197.358 78.74 90)
-      (effects (font (size 1.27 1.27)) hide)
-    )
-    (property "Datasheet" "~" (id 3) (at 195.58 78.74 0)
-      (effects (font (size 1.27 1.27)) hide)
-    )
-    (property "LCSC" "C25918" (id 4) (at 195.58 78.74 0)
-      (effects (font (size 1.27 1.27)) hide)
-    )
-    (pin "1")
-    (pin "2")
-  )
   (sheet (at 73.66 69.85) (size 27.94 30.48) (fields_autoplaced)
     (stroke (width 0.1524) (type solid) (color 0 0 0 0))
@@
     )
   )
+  (sheet (at 190.5 38.1) (size 25.4 38.1) (fields_autoplaced)
+    (stroke (width 0.1524) (type solid) (color 0 0 0 0))
+    (fill (color 0 0 0 0.0000))
+    (property "Sheet name" "LCB" (id 0) (at 190.5 37.3884 0)
+      (effects (font (size 1.27 1.27)) (justify left bottom))
+    )
+    (property "Sheet file" "LanternCommunicationBus.kicad_sch" (id 1) (at 190.5 76.7846 0)
+      (effects (font (size 1.27 1.27)) (justify left top))
+    )
+  )
