File: hw/RB3203/PowerManager.kicad_sch (KiCad schematic)
At the start: 24 parts

Commit message: Wip
Parts:
- added R?: 10k, Capacitor_SMD:C_0201_0603Metric, symbol Device:R
Connections:
- net 3V3: now also R?.2
- net BUTTON_ON: now also R?.1
Other:
- sheet Power0 ports: added 5V-A, 5V-B, EN-5V-A, EN-5V-B; removed 5V, SHUTDOWN_5V
- moved on the sheet: Q?, R?

Commit message: Wip
Parts:
- C?: value 2.2uF -> 2.2u
- C?: value 100nF -> 100n
Changed lines of the file:
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@@
       (effects (font (size 1.27 1.27)) (justify left))
     )
-    (property "Value" "2.2uF" (id 1) (at 166.37 118.11 0)
+    (property "Value" "2.2u" (id 1) (at 166.37 118.11 0)
       (effects (font (size 1.27 1.27)) (justify left))
     )
@@
     (in_bom yes) (on_board yes)
     (property "Reference" "C?" (id 0) (at 137.16 96.52 90))
-    (property "Value" "100nF" (id 1) (at 137.16 104.14 90))
+    (property "Value" "100n" (id 1) (at 137.16 104.14 90))
     (property "Footprint" "Capacitor_SMD:C_0402_1005Metric" (id 2) (at 140.97 99.3648 0)
       (effects (font (size 1.27 1.27)) hide)
